File: Start Building/Circuit Board Files/EVE-PCB/DAC1.sch (KiCad schematic (older format))
At the start: 17 parts, among them Q1 ULN2803ADWR, Q2 ULN2803ADWR, U5 MCP23017T-E_SO

Commit message: PCB Updates
Parts:
- D1, D2, D3, D4, D5, D6, D7, D8: symbol Diode:BAT43 -> EVE-PCB-rescue:BAT43-Diode
- R10, R11, R12, R13: symbol Device:R -> EVE-PCB-rescue:R-Device
Changed lines of the file:
@@
 EESchema Schematic File Version 4
-LIBS:EVE-PCB-cache
-EELAYER 26 0
+EELAYER 30 0
 EELAYER END
 $Descr A4 11693 8268
@@
 $EndComp
 $Comp
-L power:GND #PWR?
+L EVE-PCB-rescue:GND-power #PWR?
 U 1 1 5CA9821A
 P 3100 4700
@@
 Connection ~ 1550 3300
 $Comp
-L power:GND #PWR?
+L EVE-PCB-rescue:GND-power #PWR?
 U 1 1 5CA98225
 P 1050 3300
@@
 	1050 3300 1550 3300
 $Comp
-L power:+5V #PWR?
+L EVE-PCB-rescue:+5V-power #PWR?
 U 1 1 5CB343B8
 P 800 3500
@@
 	2950 4700 3100 4700
 $Comp
-L power:+5V #PWR?
+L EVE-PCB-rescue:+5V-power #PWR?
 U 1 1 5CB346D2
 P 3100 2900
@@
 NoConn ~ 4600 3350
 $Comp
-L power:+12V #PWR011
+L EVE-PCB-rescue:+12V-power #PWR011
 U 1 1 5CB549FF
 P 5950 3450
@@
 	5950 3450 5600 3450
 $Comp
-L power:GND #PWR?
+L EVE-PCB-rescue:GND-power #PWR?
 U 1 1 5CB54F53
 P 4200 3450
@@
 FAN1_POS
 $Comp
-L power:+12V #PWR04
+L EVE-PCB-rescue:+12V-power #PWR04
 U 1 1 5CB5F5B6
 P 2600 1000
@@
 A_DRUGS1
 $Comp
-L Device:R R11
+L EVE-PCB-rescue:R-Device R11
 U 1 1 5CB6FCFC
 P 5150 1800
@@
 	5300 1800 5800 1800
 $Comp
-L Diode:BAT43 D4
+L EVE-PCB-rescue:BAT43-Diode D4
 U 1 1 5CB8FF05
 P 8350 2000
@@
 WASTE1_NEG
 $Comp
-L power:+12V #PWR013
+L EVE-PCB-rescue:+12V-power #PWR013
 U 1 1 5CB9FE50
 P 8000 900
@@
 $EndComp
 $Comp
-L Diode:BAT43 D3
+L EVE-PCB-rescue:BAT43-Diode D3
 U 1 1 5CB9FE57
 P 8350 1650
@@
 	8500 2000 9000 2000
 $Comp
-L Diode:BAT43 D2
+L EVE-PCB-rescue:BAT43-Diode D2
 U 1 1 5CBAC3A9
 P 8350 1300
@@
 $EndComp
 $Comp
-L Diode:BAT43 D1
+L EVE-PCB-rescue:BAT43-Diode D1
 U 1 1 5CBAEDCC
 P 8350 950
@@
 	9000 950  8500 950
 $Comp
-L Device:R R10
+L EVE-PCB-rescue:R-Device R10
 U 1 1 5CBC545D
 P 5150 1500
@@
 	4450 800  5800 800
 $Comp
-L Diode:BAT43 D8
+L EVE-PCB-rescue:BAT43-Diode D8
 U 1 1 5CBD943B
 P 9800 2000
@@
 WASTE2_NEG
 $Comp
-L power:+12V #PWR014
+L EVE-PCB-rescue:+12V-power #PWR014
 U 1 1 5CBD9446
 P 9450 900
@@
 $EndComp
 $Comp
-L Diode:BAT43 D7
+L EVE-PCB-rescue:BAT43-Diode D7
 U 1 1 5CBD944C
 P 9800 1650
@@
 	9950 2000 10450 2000
 $Comp
-L Diode:BAT43 D6
+L EVE-PCB-rescue:BAT43-Diode D6
 U 1 1 5CBD9454
 P 9800 1300
@@
 $EndComp
 $Comp
-L Diode:BAT43 D5
+L EVE-PCB-rescue:BAT43-Diode D5
 U 1 1 5CBD945B
 P 9800 950
@@
 A_DRUGS2
 $Comp
-L Device:R R13
+L EVE-PCB-rescue:R-Device R13
 U 1 1 5CBDAD58
 P 6900 1800
@@
 	6750 1800 6200 1800
 $Comp
-L Device:R R12
+L EVE-PCB-rescue:R-Device R12
 U 1 1 5CBDAD61
 P 6900 1500
@@
 FAN2_POS
 $Comp
-L power:+12V #PWR07
+L EVE-PCB-rescue:+12V-power #PWR07
 U 1 1 5CBDEDD4
 P 3550 1000
@@
 NoConn ~ 4600 5000
 $Comp
-L power:+12V #PWR012
+L EVE-PCB-rescue:+12V-power #PWR012
 U 1 1 5CC2A1A2
 P 5950 5100
@@
 	5950 5100 5600 5100
 $Comp
-L power:GND #PWR?
+L EVE-PCB-rescue:GND-power #PWR?
 U 1 1 5CC2A1A9
 P 4200 5100
@@
 PD1_POS
 $Comp
-L power:GND #PWR05
+L EVE-PCB-rescue:GND-power #PWR05
 U 1 1 5CCCBCCC
 P 2600 1750
@@
 PD2_POS
 $Comp
-L power:GND #PWR08
+L EVE-PCB-rescue:GND-power #PWR08
 U 1 1 5CCEE678
 P 3550 1750
