File: Start Building/Circuit Board Files/EVE-PCB/DAC2.sch (KiCad schematic (older format))
At the start: 17 parts, among them Q3 ULN2803ADWR, Q4 ULN2803ADWR, U6 MCP23017T-E_SO

Commit message: PCB Updates
Parts:
- D10, D11, D12, D13, D14, D15, D16, D9: symbol Diode:BAT43 -> EVE-PCB-rescue:BAT43-Diode
- R14, R15, R16, R17: symbol Device:R -> EVE-PCB-rescue:R-Device
Connections:
- net FAN4_POS is gone; now on net +12V: L4.10
- net LED4_POS is gone; now on net +12V: L4.11
- net MEDIA4_POS is gone; now on net +12V: L4.8
- net PD4_POS is gone; now on net GND: L4.12
- net WASTE4_POS is gone; now on net +12V: L4.9
- net +5V: now also U6.15 (A0)
- net GND: no longer U6.15 (A0)
Changed lines of the file:
@@
 EESchema Schematic File Version 4
-LIBS:EVE-PCB-cache
-EELAYER 26 0
+EELAYER 30 0
 EELAYER END
 $Descr A4 11693 8268
@@
 $EndDescr
 $Comp
-L MCP23017T-E_SO:MCP23017T-E_SO U?
-U 1 1 5CD88604
-P 2400 3950
-AR Path="/5CD88604" Ref="U?"  Part="1"
-AR Path="/5CB20BFC/5CD88604" Ref="U?"  Part="1"
-AR Path="/5CA7DFAE/5CD88604" Ref="U?"  Part="1"
-AR Path="/5CA80A88/5CD88604" Ref="U6"  Part="1"
-F 0 "U6" H 2400 5117 50  0000 C CNN
-F 1 "MCP23017T-E_SO" H 2400 5026 50  0000 C CNN
-F 2 "MCP23017T-E_SO:SOIC127P1030X265-28N" H 2400 3950 50  0001 L BNN
-F 3 "Microchip" H 2400 3950 50  0001 L BNN
-F 4 "MCP23017T-E/SOCT-ND" H 2400 3950 50  0001 L BNN "Field4"
-F 5 "16-bit Input/Output Expander, I2C interface, Pb-free28 SOIC .300in T/R" H 2400 3950 50  0001 L BNN "Field5"
-F 6 "https://www.digikey.com/product-detail/en/microchip-technology/MCP23017T-E-SO/MCP23017T-E-SOCT-ND/5358289?utm_source=snapeda&utm_medium=aggregator&utm_campaign=symbol" H 2400 3950 50  0001 L BNN "Field6"
-F 7 "SOIC-28 Microchip" H 2400 3950 50  0001 L BNN "Field7"
-F 8 "MCP23017T-E/SO" H 2400 3950 50  0001 L BNN "Field8"
-	1    2400 3950
-	1    0    0    -1
-$EndComp
-$Comp
-L power:GND #PWR?
+L EVE-PCB-rescue:GND-power #PWR?
 U 1 1 5CD8860B
 P 3250 4850
@@
 NoConn ~ 3100 3350
 Wire Wire Line
-	1700 3350 1700 3450
-Wire Wire Line
 	1700 3450 1700 3550
 Connection ~ 1700 3450
 $Comp
-L power:GND #PWR?
+L EVE-PCB-rescue:GND-power #PWR?
 U 1 1 5CD88616
 P 1200 3450
@@
 	1200 3450 1700 3450
 $Comp
-L power:+5V #PWR?
+L EVE-PCB-rescue:+5V-power #PWR?
 U 1 1 5CD88623
-P 950 3650
+P 900 3250
 AR Path="/5CD88623" Ref="#PWR?"  Part="1"
 AR Path="/5CA7DFAE/5CD88623" Ref="#PWR?"  Part="1"
 AR Path="/5CA80A88/5CD88623" Ref="#PWR015"  Part="1"
-F 0 "#PWR015" H 950 3500 50  0001 C CNN
-F 1 "+5V" H 965 3823 50  0000 C CNN
-F 2 "" H 950 3650 50  0001 C CNN
-F 3 "" H 950 3650 50  0001 C CNN
-	1    950  3650
-	1    0    0    -1
-$EndComp
-Wire Wire Line
-	1700 3650 1400 3650
+F 0 "#PWR015" H 900 3100 50  0001 C CNN
+F 1 "+5V" H 915 3423 50  0000 C CNN
+F 2 "" H 900 3250 50  0001 C CNN
+F 3 "" H 900 3250 50  0001 C CNN
+	1    900  3250
+	1    0    0    -1
+$EndComp
 Wire Wire Line
 	3100 4850 3250 4850
 $Comp
-L power:+5V #PWR?
+L EVE-PCB-rescue:+5V-power #PWR?
 U 1 1 5CD8862B
 P 3250 3050
@@
 NoConn ~ 4750 3500
 $Comp
-L power:+12V #PWR?
+L EVE-PCB-rescue:+12V-power #PWR?
 U 1 1 5CD8866E
 P 6100 3600
@@
 	6100 3600 5750 3600
 $Comp
-L power:GND #PWR?
+L EVE-PCB-rescue:GND-power #PWR?
 U 1 1 5CD88675
 P 4350 3600
@@
 FAN3_POS
 $Comp
-L power:+12V #PWR?
+L EVE-PCB-rescue:+12V-power #PWR?
 U 1 1 5CD8868C
 P 2750 1150
@@
 A_DRUGS3
 $Comp
-L Device:R R?
+L EVE-PCB-rescue:R-Device R?
 U 1 1 5CD886A7
 P 5300 1950
@@
 	5450 1950 5950 1950
 $Comp
-L Diode:BAT43 D?
+L EVE-PCB-rescue:BAT43-Diode D?
 U 1 1 5CD886AF
 P 8500 2150
@@
 WASTE3_NEG
 $Comp
-L power:+12V #PWR?
+L EVE-PCB-rescue:+12V-power #PWR?
 U 1 1 5CD886BB
 P 8150 1050
@@
 $EndComp
 $Comp
-L Diode:BAT43 D?
+L EVE-PCB-rescue:BAT43-Diode D?
 U 1 1 5CD886C1
 P 8500 1800
@@
 	8650 2150 9150 2150
 $Comp
-L Diode:BAT43 D?
+L EVE-PCB-rescue:BAT43-Diode D?
 U 1 1 5CD886C9
 P 8500 1450
@@
 $EndComp
 $Comp
-L Diode:BAT43 D?
+L EVE-PCB-rescue:BAT43-Diode D?
 U 1 1 5CD886D0
 P 8500 1100
@@
 	9150 1100 8650 1100
 $Comp
-L Device:R R?
+L EVE-PCB-rescue:R-Device R?
 U 1 1 5CD886E5
 P 5300 1650
@@
 	4600 950  5950 950
 $Comp
-L Diode:BAT43 D?
+L EVE-PCB-rescue:BAT43-Diode D?
 U 1 1 5CD886F2
 P 9950 2150
@@
 WASTE4_NEG
 $Comp
-L power:+12V #PWR?
+L EVE-PCB-rescue:+12V-power #PWR?
 U 1 1 5CD886FD
 P 9600 1050
@@
 $EndComp
 $Comp
-L Diode:BAT43 D?
+L EVE-PCB-rescue:BAT43-Diode D?
 U 1 1 5CD88703
 P 9950 1800
@@
 	10100 2150 10600 2150
 $Comp
-L Diode:BAT43 D?
+L EVE-PCB-rescue:BAT43-Diode D?
 U 1 1 5CD8870B
 P 9950 1450
@@
 $EndComp
 $Comp
-L Diode:BAT43 D?
+L EVE-PCB-rescue:BAT43-Diode D?
 U 1 1 5CD88712
 P 9950 1100
@@
 A_DRUGS4
 $Comp
-L Device:R R?
+L EVE-PCB-rescue:R-Device R?
 U 1 1 5CD88733
 P 7050 1950
@@
 	6900 1950 6350 1950
 $Comp
-L Device:R R?
+L EVE-PCB-rescue:R-Device R?
 U 1 1 5CD8873C
 P 7050 1650
@@
 DRUG4_POS
 Text Label 4200 1400 2    50   ~ 0
-MEDIA2_POS
+MEDIA4_POS
 Text Label 4200 1500 2    50   ~ 0
-WASTE2_POS
+WASTE4_POS
 Text Label 4200 1600 2    50   ~ 0
-LED2_POS
+LED4_POS
 Text Label 4200 1700 2    50   ~ 0
-FAN2_POS
-$Comp
-L power:+12V #PWR?
+FAN4_POS
+$Comp
+L EVE-PCB-rescue:+12V-power #PWR?
 U 1 1 5CD8874E
 P 3700 1150
@@
 NoConn ~ 1700 4550
 Wire Wire Line
-	1400 3650 1400 3750
-Wire Wire Line
-	1400 3750 950  3750
-Wire Wire Line
-	950  3750 950  3650
+	900  3350 900  3250
 Wire Wire Line
 	1300 3850 1700 3850
@@
 NoConn ~ 4750 5150
 $Comp
-L power:+12V #PWR?
+L EVE-PCB-rescue:+12V-power #PWR?
 U 1 1 5CD887A9
 P 6100 5250
@@
 	6100 5250 5750 5250
 $Comp
-L power:GND #PWR?
+L EVE-PCB-rescue:GND-power #PWR?
 U 1 1 5CD887B0
 P 4350 5250
@@
 PD3_POS
 $Comp
-L power:GND #PWR?
+L EVE-PCB-rescue:GND-power #PWR?
 U 1 1 5CD887EE
 P 2750 1900
@@
 	2750 1900 3250 1900
 Text Label 4200 1900 2    50   ~ 0
-PD2_POS
-$Comp
-L power:GND #PWR?
+PD4_POS
+$Comp
+L EVE-PCB-rescue:GND-power #PWR?
 U 1 1 5CD887F6
 P 3700 1900
@@
 Wire Wire Line
 	3500 4350 3100 4350
+$Comp
+L MCP23017T-E_SO:MCP23017T-E_SO U?
+U 1 1 5CD88604
+P 2400 3950
+AR Path="/5CD88604" Ref="U?"  Part="1"
+AR Path="/5CB20BFC/5CD88604" Ref="U?"  Part="1"
+AR Path="/5CA7DFAE/5CD88604" Ref="U?"  Part="1"
+AR Path="/5CA80A88/5CD88604" Ref="U6"  Part="1"
+F 0 "U6" H 2400 5117 50  0000 C CNN
+F 1 "MCP23017T-E_SO" H 2400 5026 50  0000 C CNN
+F 2 "MCP23017T-E_SO:SOIC127P1030X265-28N" H 2400 3950 50  0001 L BNN
+F 3 "Microchip" H 2400 3950 50  0001 L BNN
+F 4 "MCP23017T-E/SOCT-ND" H 2400 3950 50  0001 L BNN "Field4"
+F 5 "16-bit Input/Output Expander, I2C interface, Pb-free28 SOIC .300in T/R" H 2400 3950 50  0001 L BNN "Field5"
+F 6 "https://www.digikey.com/product-detail/en/microchip-technology/MCP23017T-E-SO/MCP23017T-E-SOCT-ND/5358289?utm_source=snapeda&utm_medium=aggregator&utm_campaign=symbol" H 2400 3950 50  0001 L BNN "Field6"
+F 7 "SOIC-28 Microchip" H 2400 3950 50  0001 L BNN "Field7"
+F 8 "MCP23017T-E/SO" H 2400 3950 50  0001 L BNN "Field8"
+	1    2400 3950
+	1    0    0    -1
+$EndComp
+Wire Wire Line
+	1700 3650 1400 3650
+Wire Wire Line
+	1700 3350 900  3350
+Connection ~ 900  3350
+Wire Wire Line
+	1400 3650 1400 3700
+Wire Wire Line
+	1400 3700 900  3700
+Wire Wire Line
+	900  3700 900  3350
 $EndSCHEMATC
