File: Start Building/Circuit Board Files/EVE-PCB/EVE-PCB.sch (KiCad schematic (older format))
At the start: 20 parts, among them J1 Raspberry_Pi_2_3, J2 PJ-002A, Q5 UA7805CKCT, U1 ADS1015IDGSR, U2 LM324DR, U3 BSN20BKR, U4 BSN20BKR

Commit message: PCB Updates
Parts:
- C1, C2, C3: symbol Device:C -> EVE-PCB-rescue:C-Device
- D17: symbol Device:D -> EVE-PCB-rescue:D-Device
- J1: symbol Connector:Raspberry_Pi_2_3 -> EVE-PCB-rescue:Raspberry_Pi_2_3-Connector
- R1, R2, R3, R4, R5, R6, R7, R8, R9: symbol Device:R -> EVE-PCB-rescue:R-Device
Changed lines of the file:
@@
 EESchema Schematic File Version 4
-LIBS:EVE-PCB-cache
-EELAYER 26 0
+EELAYER 30 0
 EELAYER END
 $Descr A4 11693 8268
@@
 SCL
 $Comp
-L power:GND #PWR0101
+L EVE-PCB-rescue:GND-power #PWR0101
 U 1 1 5CAF017E
 P 3250 1950
@@
 PD4_NEG
 $Comp
-L Device:R R1
+L EVE-PCB-rescue:R-Device R1
 U 1 1 5CAF996E
 P 7700 1150
@@
 AIN3
 $Comp
-L Device:R R2
+L EVE-PCB-rescue:R-Device R2
 U 1 1 5CAFA8CC
 P 7700 1550
@@
 $EndComp
 $Comp
-L Device:R R3
+L EVE-PCB-rescue:R-Device R3
 U 1 1 5CAFB32D
 P 7700 1950
@@
 $EndComp
 $Comp
-L Device:R R4
+L EVE-PCB-rescue:R-Device R4
 U 1 1 5CAFB4DE
 P 7700 2350
@@
 $EndComp
 $Comp
-L power:GND #PWR0102
+L EVE-PCB-rescue:GND-power #PWR0102
 U 1 1 5CB02683
 P 4900 2400
@@
 $EndComp
 $Comp
-L power:GND #PWR0103
+L EVE-PCB-rescue:GND-power #PWR0103
 U 1 1 5CB0A15A
 P 1550 1150
@@
 $EndComp
 $Comp
-L Device:R R5
+L EVE-PCB-rescue:R-Device R5
 U 1 1 5CB13406
 P 10000 1300
@@
 	9900 1100 10000 1100
 $Comp
-L power:+3V3 #PWR0105
+L EVE-PCB-rescue:+3V3-power #PWR0105
 U 1 1 5CB13B9F
 P 10400 1500
@@
 SCL
 $Comp
-L power:+5V #PWR0106
+L EVE-PCB-rescue:+5V-power #PWR0106
 U 1 1 5CB15101
 P 9000 1500
@@
 $EndComp
 $Comp
-L Device:R R6
+L EVE-PCB-rescue:R-Device R6
 U 1 1 5CB15AFC
 P 9400 1300
@@
 	3200 1050 3200 900
 $Comp
-L Device:R R7
+L EVE-PCB-rescue:R-Device R7
 U 1 1 5CB348CD
 P 3550 1700
@@
 $EndComp
 $Comp
-L Device:R R9
+L EVE-PCB-rescue:R-Device R9
 U 1 1 5CB4AB1F
 P 10000 2150
@@
 	9900 1950 10000 1950
 $Comp
-L power:+3V3 #PWR0108
+L EVE-PCB-rescue:+3V3-power #PWR0108
 U 1 1 5CB4AB28
 P 10400 2350
@@
 SDA
 $Comp
-L power:+5V #PWR0109
+L EVE-PCB-rescue:+5V-power #PWR0109
 U 1 1 5CB4AB37
 P 9000 2350
@@
 $EndComp
 $Comp
-L Device:R R8
+L EVE-PCB-rescue:R-Device R8
 U 1 1 5CB4AB3D
 P 9400 2150
@@
 	9100 1950 9400 1950
 $Comp
-L power:+5V #PWR0111
+L EVE-PCB-rescue:+5V-power #PWR0111
 U 1 1 5CAD3B2B
 P 4900 1100
@@
 $EndComp
 $Comp
-L power:+5V #PWR0112
+L EVE-PCB-rescue:+5V-power #PWR0112
 U 1 1 5CAD789A
 P 3800 1700
@@
 $EndComp
 $Comp
-L power:+5V #PWR0113
+L EVE-PCB-rescue:+5V-power #PWR0113
 U 1 1 5CADB22B
 P 3200 900
@@
 $EndComp
 $Comp
-L Connector:Raspberry_Pi_2_3 J1
+L EVE-PCB-rescue:Raspberry_Pi_2_3-Connector J1
 U 1 1 5CAE0D0F
 P 6150 4350
@@
 $EndComp
 $Comp
-L power:+3V3 #PWR02
+L EVE-PCB-rescue:+3V3-power #PWR02
 U 1 1 5CAE0D83
 P 7050 3050
@@
 Connection ~ 6350 3050
 $Comp
-L power:GND #PWR01
+L EVE-PCB-rescue:GND-power #PWR01
 U 1 1 5CB31D3A
 P 7000 5700
@@
 $EndComp
 $Comp
-L power:GND #PWR0104
+L EVE-PCB-rescue:GND-power #PWR0104
 U 1 1 5CDD5CE7
 P 1750 4400
@@
 	1350 4000 1200 4000
 $Comp
-L Device:D D17
+L EVE-PCB-rescue:D-Device D17
 U 1 1 5CE0AEF1
 P 1500 3850
@@
 	2200 4300 1750 4300
 $Comp
-L power:+12V #PWR?
+L EVE-PCB-rescue:+12V-power #PWR?
 U 1 1 5CE2DC86
 P 2000 3700
@@
 	2200 4050 2200 4300
 $Comp
-L Device:C C2
+L EVE-PCB-rescue:C-Device C2
 U 1 1 5CE50296
 P 3650 4100
@@
 $EndComp
 $Comp
-L power:+5V #PWR0110
+L EVE-PCB-rescue:+5V-power #PWR0110
 U 1 1 5CE53FA4
 P 3650 3700
@@
 	3650 3700 3650 3950
 $Comp
-L Device:C C3
+L EVE-PCB-rescue:C-Device C3
 U 1 1 5CE84515
 P 4150 4100
@@
 	1650 3850 1750 3850
 $Comp
-L Device:C C1
+L EVE-PCB-rescue:C-Device C1
 U 1 1 5CAC5E05
 P 1750 4100
