File: Start Building/Circuit Board Files/EVE-PCB/_autosave-EVE-PCB-V2.kicad_pcb (KiCad board)
At the start: 2 copper layers, 103.5 x 99.5 mm, 54 parts, among them J1 Raspberry_Pi_2_3, J2 PJ-002A, Q1 DW18, Q2 DW18, Q3 DW18, Q4 DW18, Q5 TO254P465X1016X1883-3P, U1 ADS1015IDGSR, U2 LM324DR, U3 BSN20BKR, U4 BSN20BKR, U5 MCP23017T-E_SO, U6 MCP23017T-E_SO

Commit message: PCB Updates
Parts:
- L1, L2, L3, L4: value SHDR12W60P935X350_2X6_2250X1800X2420P -> 1841539
- Q1, Q2, Q3, Q4: value DW18 -> ULN2803ADWR
- Q5: value TO254P465X1016X1883-3P -> UA7805CKCT
- moved R14 33.0 mm to (124.5, 94.5), turned to 270 degrees
- moved R12 22.1 mm to (157.0, 94.5), turned to 270 degrees
- moved R10 19.7 mm to (179.8, 94.5), turned to 270 degrees
- moved R16 19.4 mm to (107.2, 94.5), turned to 270 degrees
- moved R17 16.1 mm to (106.2, 84.3), turned to 270 degrees
- moved R2 15.4 mm to (131.7, 75.7), turned to 180 degrees
- moved R6 15.3 mm to (146.6, 79.8)
- moved R13 11.3 mm to (165.1, 84.3), turned to 270 degrees
- moved D3 11.2 mm to (111.6, 38.7)
- moved D5 11.2 mm to (105.0, 47.8)
- moved R15 8.64 mm to (111.3, 82.6), turned to 90 degrees
- moved R11 8.08 mm to (172.7, 82.8), turned to 90 degrees
- moved U3 7.07 mm to (165.2, 61.4), turned to 180 degrees
- moved Q1 6.62 mm to (180.8, 83.3), turned to 180 degrees
- moved Q2 6.62 mm to (156.6, 83.6)
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Connections:
- U6 pad 15: GND -> +5V
Routing:
- net /DAC1/A_DRUGS2: track 0.00 -> 151.1 mm, vias 0 -> 2
- net /DAC1/A_DRUGS1: track 0.00 -> 142.0 mm, vias 0 -> 2
- net +12V: track 0.00 -> 140.4 mm, vias 0 -> 9
- net /DAC1/A_SFAN1: track 0.00 -> 138.0 mm, vias 0 -> 2
- net /SCL: track 0.00 -> 137.4 mm, vias 0 -> 5
- net /DAC1/A_MEDIA1: track 0.00 -> 136.8 mm, vias 0 -> 2
- net /DAC1/A_SFAN2: track 0.00 -> 135.5 mm, vias 0 -> 2
- net /SDA: track 0.00 -> 128.3 mm, vias 0 -> 5
- net /DAC1/A_WASTE2: track 0.00 -> 121.5 mm, vias 0 -> 2
- net /DAC1/A_WASTE1: track 0.00 -> 121.2 mm, vias 0 -> 2
- net +3V3: track 0.00 -> 119.5 mm, vias 0 -> 2
- net /DAC1/A_MEDIA2: track 0.00 -> 110.7 mm, vias 0 -> 2
- net GND: track 0.00 -> 104.2 mm, vias 0 -> 4
- net /DAC2/A_WASTE3: track 0.00 -> 92.9 mm, vias 0 -> 2
- net /DAC2/A_SFAN3: track 0.00 -> 81.7 mm, vias 0 -> 2
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- added copper zone on B.Cu, net +12V
- added copper zone on In2.Cu, net +5V
- added copper zone on F.Cu, net GND
- added copper zone on In1.Cu, net GND
Other:
- copper layers 2 -> 4
- net class 12v added: clearance 0.6, trace_width 0.5, via_dia 0.8, via_drill 0.4
- net class 5v added: clearance 0.2, trace_width 0.25, via_dia 0.8, via_drill 0.4
