File: Start Building/Circuit Board Files/EVE-PCB/v5/v5_proj/DAC1.sch (KiCad schematic (older format))
At the start: 10 parts

Commit message: Finalize schematic
Parts:
- R20, R21: value 50Ω -> 2Ω; LCSC C25487 -> C49298
Changed lines of the file:
@@
 P 5150 1500
 F 0 "R20" V 4943 1500 50  0000 C CNN
-F 1 "50Ω" V 5034 1500 50  0000 C CNN
+F 1 "2Ω" V 5034 1500 50  0000 C CNN
 F 2 "Resistor_SMD:R_2512_6332Metric" V 5080 1500 50  0001 C CNN
-F 3 "25121WF499JT4E" H 5150 1500 50  0001 C CNN
-F 4 "C25487" H 5150 1500 50  0001 C CNN "LCSC"
+F 3 "25121WF200KT4E" H 5150 1500 50  0001 C CNN
+F 4 "C49298" H 5150 1500 50  0001 C CNN "LCSC"
 F 5 "2512" H 5150 1500 50  0001 C CNN "Package"
 F 6 "1.05" H 5150 1500 50  0001 C CNN "Power"
@@
 P 6900 1500
 F 0 "R21" V 6693 1500 50  0000 C CNN
-F 1 "50Ω" V 6784 1500 50  0000 C CNN
+F 1 "2Ω" V 6784 1500 50  0000 C CNN
 F 2 "Resistor_SMD:R_2512_6332Metric" V 6830 1500 50  0001 C CNN
-F 3 "25121WF499JT4E" H 6900 1500 50  0001 C CNN
-F 4 "C25487" H 6900 1500 50  0001 C CNN "LCSC"
+F 3 "25121WF200KT4E" H 6900 1500 50  0001 C CNN
+F 4 "C49298" H 6900 1500 50  0001 C CNN "LCSC"
 F 5 "2512" H 6900 1500 50  0001 C CNN "Package"
 F 6 "1.05" H 6900 1500 50  0001 C CNN "Power"
