File: Start Building/Circuit Board Files/EVE-PCB/v5/v5_proj/DAC2.sch (KiCad schematic (older format))
At the start: 26 parts, among them Q10 DMN6140LQ-7, Q11 DMN6140LQ-7, Q4 ULN2803ADWR, Q5 ULN2803ADWR, U8 MCP23017-E/SO

Commit message: Finalize schematic
Parts:
- R24, R25: value 50Ω -> 2Ω; LCSC C25487 -> C49298
Changed lines of the file:
@@
 AR Path="/5CA80A88/5CD886E5" Ref="R24"  Part="1"
 F 0 "R24" V 5093 1650 50  0000 C CNN
-F 1 "50Ω" V 5184 1650 50  0000 C CNN
+F 1 "2Ω" V 5184 1650 50  0000 C CNN
 F 2 "Resistor_SMD:R_2512_6332Metric" V 5230 1650 50  0001 C CNN
-F 3 "25121WF499JT4E" H 5300 1650 50  0001 C CNN
-F 4 "C25487" H 5300 1650 50  0001 C CNN "LCSC"
+F 3 "25121WF200KT4E" H 5300 1650 50  0001 C CNN
+F 4 "C49298" H 5300 1650 50  0001 C CNN "LCSC"
 F 5 "2512" H 5300 1650 50  0001 C CNN "Package"
 F 6 "1.05" H 5300 1650 50  0001 C CNN "Power"
@@
 AR Path="/5CA80A88/5CD8873C" Ref="R25"  Part="1"
 F 0 "R25" V 6843 1650 50  0000 C CNN
-F 1 "50Ω" V 6934 1650 50  0000 C CNN
+F 1 "2Ω" V 6934 1650 50  0000 C CNN
 F 2 "Resistor_SMD:R_2512_6332Metric" V 6980 1650 50  0001 C CNN
-F 3 "25121WF499JT4E" H 7050 1650 50  0001 C CNN
-F 4 "C25487" H 7050 1650 50  0001 C CNN "LCSC"
+F 3 "25121WF200KT4E" H 7050 1650 50  0001 C CNN
+F 4 "C49298" H 7050 1650 50  0001 C CNN "LCSC"
 F 5 "2512" H 7050 1650 50  0001 C CNN "Package"
 F 6 "1.05" H 7050 1650 50  0001 C CNN "Power"
