File: Start Building/Circuit Board Files/EVE-PCB/v5/v5_proj/EVE-PCB-V4.kicad_pcb (KiCad board)
At the start: 4 copper layers, 103.5 x 90.6 mm, 102 parts, among them J1 PJ-102AH, J2 2x20 Male Header, J3 1725669, Q1 UA7805CKCT, Q10 DMN6140LQ-7, Q11 DMN6140LQ-7, Q12 DMN6140LQ-7, Q2 ULN2803ADWR, Q3 ULN2803ADWR, Q4 ULN2803ADWR, Q5 ULN2803ADWR, Q6 DMN6140LQ-7, Q7 DMN6140LQ-7, Q8 DMN6140LQ-7, Q9 DMN6140LQ-7, U1 PCA9685PW, U2 ADS1115IDGSR, U3 TLV4314IPWR, U4 TLV4314IPWR, U5 MCP1501-10E/SN, U7 MCP23017-E/SO, U8 MCP23017-E/SO

Commit message: Finalize schematic
Parts:
- added C22: 0.1μF, Capacitor_SMD:C_0402_1005Metric, F.Cu at (375.6, 102.5)
- added C23: 0.1μF, Capacitor_SMD:C_0402_1005Metric, F.Cu at (386.6, 91.2)
- added C24: 10pF, Capacitor_SMD:C_0402_1005Metric, F.Cu at (382.2, 95.2)
- added C25: 10pF, Capacitor_SMD:C_0402_1005Metric, F.Cu at (419.7, 58.1)
- added C26: 10pF, Capacitor_SMD:C_0402_1005Metric, F.Cu at (428.5, 48.9)
- added C27: 10pF, Capacitor_SMD:C_0402_1005Metric, F.Cu at (402.8, 74.5)
- added C28: 0.1μF, Capacitor_SMD:C_0402_1005Metric, F.Cu at (387.7, 89.2)
- added C29: 0.1μF, Capacitor_SMD:C_0402_1005Metric, F.Cu at (395.0, 81.8)
- added C30: 0.1μF, Capacitor_SMD:C_0402_1005Metric, F.Cu at (428.5, 47.0)
- added C31: 0.1μF, Capacitor_SMD:C_0402_1005Metric, F.Cu at (406.2, 72.4)
- added C32: 0.1μF, Capacitor_SMD:C_0402_1005Metric, F.Cu at (419.7, 60.1)
- added C33: 2.2μF, Capacitor_SMD:C_0603_1608Metric, F.Cu at (385.7, 82.5)
- added C34: 2.2μF, Capacitor_SMD:C_0603_1608Metric, F.Cu at (385.7, 85.0)
- added C35: 0.1μF, Capacitor_SMD:C_0402_1005Metric, F.Cu at (409.0, 69.9)
- added C36: 0.1μF, Capacitor_SMD:C_0402_1005Metric, F.Cu at (379.5, 100.0)
- added C37: 0.1μF, Capacitor_SMD:C_0402_1005Metric, F.Cu at (415.2, 64.1)
- added C38: 0.1μF, Capacitor_SMD:C_0402_1005Metric, F.Cu at (401.7, 77.3)
- added C39: 0.1μF, Capacitor_SMD:C_0402_1005Metric, F.Cu at (424.1, 53.2)
- added C40: 0.1μF, Capacitor_SMD:C_0402_1005Metric, F.Cu at (416.7, 62.1)
- added C41: 0.1μF, Capacitor_SMD:C_0402_1005Metric, F.Cu at (385.1, 93.2)
- added C42: 0.1μF, Capacitor_SMD:C_0402_1005Metric, F.Cu at (422.6, 55.2)
- added C43: 2.2μF, Capacitor_SMD:C_0603_1608Metric, F.Cu at (426.6, 44.4)
- added C44: 2.2μF, Capacitor_SMD:C_0603_1608Metric, F.Cu at (422.2, 49.0)
- added C45: 0.1μF, Capacitor_SMD:C_0402_1005Metric, F.Cu at (422.6, 57.2)
- added C46: 2.2μF, Capacitor_SMD:C_0603_1608Metric, F.Cu at (396.5, 75.6)
- added C47: 2.2μF, Capacitor_SMD:C_0603_1608Metric, F.Cu at (370.3, 100.2)
- added C48: 2.2μF, Capacitor_SMD:C_0603_1608Metric, F.Cu at (422.2, 46.5)
- added C49: 2.2μF, Capacitor_SMD:C_0603_1608Metric, F.Cu at (426.6, 41.9)
- added D2: PMEG6010CEH, Diode_SMD:D_SOD-123F, F.Cu at (377.2, 79.2)
- added D25: PMEG6010CEH, Diode_SMD:D_SOD-123F, F.Cu at (408.2, 49.2)
- added D26: PMEG6010CEH, Diode_SMD:D_SOD-123F, F.Cu at (413.8, 42.3)
- added D27: PMEG6010CEH, Diode_SMD:D_SOD-123F, F.Cu at (349.3, 102.8)
- added D28: PMEG6010CEH, Diode_SMD:D_SOD-123F, F.Cu at (422.4, 34.4)
- added D29: PMEG6010CEH, Diode_SMD:D_SOD-123F, F.Cu at (389.0, 67.5)
- added D30: PMEG6010CEH, Diode_SMD:D_SOD-123F, F.Cu at (356.7, 97.9)
- added D31: PMEG6010CEH, Diode_SMD:D_SOD-123F, F.Cu at (383.5, 67.5)
- added D32: PMEG6010CEH, Diode_SMD:D_SOD-123F, F.Cu at (338.3, 102.6)
- added D33: PMEG6010CEH, Diode_SMD:D_SOD-123F, F.Cu at (392.1, 49.7)
- added D34: PMEG6010CEH, Diode_SMD:D_SOD-123F, F.Cu at (351.2, 96.1)
- added D35: PMEG6010CEH, Diode_SMD:D_SOD-123F, F.Cu at (377.4, 69.1)
- added D36: PMEG6010CEH, Diode_SMD:D_SOD-123F, F.Cu at (416.9, 34.4)
- added D37: PMEG6010CEH, Diode_SMD:D_SOD-123F, F.Cu at (377.4, 72.5)
- added D38: PMEG6010CEH, Diode_SMD:D_SOD-123F, F.Cu at (351.2, 99.5)
- added D39: PMEG6010CEH, Diode_SMD:D_SOD-123F, F.Cu at (408.4, 42.3)
- added J4: 2x20 Male Header, Connector_PinHeader_2.54mm:PinHeader_2x20_P2.54mm_Vertical, F.Cu at (49.5, 49.5)
- added J5: Conn_02x03_Odd_Even, Connector_PinHeader_2.54mm:PinHeader_2x03_P2.54mm_Vertical, F.Cu at (358.3, 50.4)
- added J6: Conn_01x18, ICs:282888-7, F.Cu at (61.0, 133.3)
- added J7: Conn_01x18, ICs:282888-7, F.Cu at (165.1, 133.3)
- added J8: Conn_01x18, ICs:282888-7, F.Cu at (113.0, 133.3)
- added J9: Conn_01x18, ICs:282888-7, F.Cu at (217.2, 133.3)
- added L5: 680uH, Inductor_SMD:L_6.3x6.3_H3, F.Cu at (401.1, 48.1)
- added L6: 680uH, Inductor_SMD:L_6.3x6.3_H3, F.Cu at (409.9, 28.8)
- added L7: 680uH, Inductor_SMD:L_6.3x6.3_H3, F.Cu at (361.8, 71.5)
- added L8: 680uH, Inductor_SMD:L_6.3x6.3_H3, F.Cu at (353.0, 84.1)
- added Q13: DMN6140LQ-7, Package_TO_SOT_SMD:SOT-23, F.Cu at (393.9, 67.5)
- added Q14: DMN6140LQ-7, Package_TO_SOT_SMD:SOT-23, F.Cu at (367.9, 96.7)
- added Q15: DMN6140LQ-7, Package_TO_SOT_SMD:SOT-23, F.Cu at (387.8, 76.0)
- added Q16: DMN6140LQ-7, Package_TO_SOT_SMD:SOT-23, F.Cu at (398.3, 62.2)
- added Q17: DMN6140LQ-7, Package_TO_SOT_SMD:SOT-23, F.Cu at (376.7, 87.8)
- added Q18: DMN6140LQ-7, Package_TO_SOT_SMD:SOT-23, F.Cu at (387.8, 71.5)
- added Q19: DMN6140LQ-7, Package_TO_SOT_SMD:SOT-23, F.Cu at (372.7, 92.3)
- added Q20: DMN6140LQ-7, Package_TO_SOT_SMD:SOT-23, F.Cu at (418.0, 46.2)
- added Q21: DMN6140LQ-7, Package_TO_SOT_SMD:SOT-23, F.Cu at (426.3, 38.4)
- added Q22: DMN6140LQ-7, Package_TO_SOT_SMD:SOT-23, F.Cu at (381.5, 83.1)
- added Q23: DMN6140LQ-7, Package_TO_SOT_SMD:SOT-23, F.Cu at (405.8, 57.7)
- added Q24: DMN6140LQ-7, Package_TO_SOT_SMD:SOT-23, F.Cu at (398.4, 66.8)
- added Q25: DMN6140LQ-7, Package_TO_SOT_SMD:SOT-23, F.Cu at (392.2, 72.0)
- added Q26: DMN6140LQ-7, Package_TO_SOT_SMD:SOT-23, F.Cu at (366.1, 101.2)
- added Q27: DMN6140LQ-7, Package_TO_SOT_SMD:SOT-23, F.Cu at (396.7, 72.0)
- added Q28: DMN6140LQ-7, Package_TO_SOT_SMD:SOT-23, F.Cu at (392.2, 76.6)
- added Q29: DMN6140LQ-7, Package_TO_SOT_SMD:SOT-23, F.Cu at (410.2, 57.7)
- added Q30: DMN6140LQ-7, Package_TO_SOT_SMD:SOT-23, F.Cu at (402.8, 62.3)
- added Q31: DMN6140LQ-7, Package_TO_SOT_SMD:SOT-23, F.Cu at (417.6, 50.9)
- added Q32: DMN6140LQ-7, Package_TO_SOT_SMD:SOT-23, F.Cu at (422.4, 42.9)
- added R33: 10KΩ, Resistor_SMD:R_0402_1005Metric, F.Cu at (400.4, 70.5)
- added R34: 10KΩ, Resistor_SMD:R_0402_1005Metric, F.Cu at (390.4, 79.8)
- added R35: 10KΩ, Resistor_SMD:R_0402_1005Metric, F.Cu at (417.1, 54.1)
- added R36: 0.4Ω, Resistor_SMD:R_2512_6332Metric, F.Cu at (353.1, 77.7)
- added R37: 0.4Ω, Resistor_SMD:R_2512_6332Metric, F.Cu at (369.0, 65.1)
- added R38: 10KΩ, Resistor_SMD:R_0402_1005Metric, F.Cu at (430.1, 41.0)
- added R39: 10KΩ, Resistor_SMD:R_0402_1005Metric, F.Cu at (389.2, 82.2)
- added R40: 10KΩ, Resistor_SMD:R_0402_1005Metric, F.Cu at (410.9, 61.0)
- added R41: 10KΩ, Resistor_SMD:R_0402_1005Metric, F.Cu at (376.0, 96.0)
- added R42: 10KΩ, Resistor_SMD:R_0402_1005Metric, F.Cu at (406.5, 65.9)
- added R43: 10KΩ, Resistor_SMD:R_0402_1005Metric, F.Cu at (413.9, 58.1)
- added R44: 10KΩ, Resistor_SMD:R_0402_1005Metric, F.Cu at (369.8, 102.4)
- added R45: 10KΩ, Resistor_SMD:R_0402_1005Metric, F.Cu at (373.8, 98.5)
- added R46: 0.4Ω, Resistor_SMD:R_2512_6332Metric, F.Cu at (344.3, 91.5)
- added R47: 0.4Ω, Resistor_SMD:R_2512_6332Metric, F.Cu at (385.0, 50.5)
- added R48: 80Ω, Resistor_SMD:R_0805_2012Metric, F.Cu at (377.1, 91.5)
- added R49: 80Ω, Resistor_SMD:R_0805_2012Metric, F.Cu at (386.7, 79.8)
- added R50: 80Ω, Resistor_SMD:R_0805_2012Metric, F.Cu at (359.7, 102.2)
- added R51: 80Ω, Resistor_SMD:R_0805_2012Metric, F.Cu at (372.3, 96.1)
- added R52: 80Ω, Resistor_SMD:R_0805_2012Metric, F.Cu at (430.7, 35.6)
- added R53: 80Ω, Resistor_SMD:R_0805_2012Metric, F.Cu at (407.2, 61.5)
- added R54: 80Ω, Resistor_SMD:R_0805_2012Metric, F.Cu at (402.8, 66.0)
- added R55: 80Ω, Resistor_SMD:R_0805_2012Metric, F.Cu at (430.7, 38.5)
- added R56: 10KΩ, Resistor_SMD:R_0402_1005Metric, F.Cu at (403.3, 72.5)
- added R57: 10KΩ, Resistor_SMD:R_0402_1005Metric, F.Cu at (392.1, 83.8)
- added R58: 20KΩ, Resistor_SMD:R_0402_1005Metric, F.Cu at (424.1, 51.2)
- added R59: 20KΩ, Resistor_SMD:R_0402_1005Metric, F.Cu at (376.7, 98.0)
- added R60: 10KΩ, Resistor_SMD:R_0402_1005Metric, F.Cu at (409.4, 65.9)
- added R61: 330KΩ, Resistor_SMD:R_0402_1005Metric, F.Cu at (403.3, 70.5)
- added R62: 330KΩ, Resistor_SMD:R_0402_1005Metric, F.Cu at (378.9, 96.0)
- added R63: 330KΩ, Resistor_SMD:R_0402_1005Metric, F.Cu at (413.9, 60.1)
- added R64: 330KΩ, Resistor_SMD:R_0402_1005Metric, F.Cu at (373.8, 100.5)
- added R65: 330KΩ, Resistor_SMD:R_0402_1005Metric, F.Cu at (413.8, 62.1)
- added R66: 330KΩ, Resistor_SMD:R_0402_1005Metric, F.Cu at (430.1, 45.0)
- added R67: 330KΩ, Resistor_SMD:R_0402_1005Metric, F.Cu at (416.8, 58.1)
- added R68: 20KΩ, Resistor_SMD:R_0402_1005Metric, F.Cu at (392.1, 81.8)
- added R69: 20KΩ, Resistor_SMD:R_0402_1005Metric, F.Cu at (416.8, 56.1)
- added R70: 20KΩ, Resistor_SMD:R_0402_1005Metric, F.Cu at (387.7, 87.3)
- added R71: 20KΩ, Resistor_SMD:R_0402_1005Metric, F.Cu at (425.6, 48.7)
- added R72: 10KΩ, Resistor_SMD:R_0402_1005Metric, F.Cu at (421.2, 53.2)
- added R73: 20KΩ, Resistor_SMD:R_0402_1005Metric, F.Cu at (399.9, 75.3)
- added R74: 20KΩ, Resistor_SMD:R_0402_1005Metric, F.Cu at (395.9, 77.8)
- added U10: INA219AxDCN, Package_TO_SOT_SMD:SOT-23-8, F.Cu at (376.9, 83.2)
- added U11: INA219AxDCN, Package_TO_SOT_SMD:SOT-23-8, F.Cu at (368.1, 92.1)
- added U12: AD5242, Package_SO:TSSOP-16_4.4x5mm_P0.65mm, F.Cu at (344.4, 85.8)
- added U13: AD5242, Package_SO:TSSOP-16_4.4x5mm_P0.65mm, F.Cu at (376.3, 51.4)
- added U14: PCA9685PW, Package_SO:TSSOP-28_4.4x9.7mm_P0.65mm, F.Cu at (157.5, 83.8)
- added U15: INA219AxDCN, Package_TO_SOT_SMD:SOT-23-8, F.Cu at (430.6, 27.2)
- added U16: INA219AxDCN, Package_TO_SOT_SMD:SOT-23-8, F.Cu at (413.3, 46.3)
- added U17: TLV4314IPWR, Package_SO:TSSOP-14_4.4x5mm_P0.65mm, F.Cu at (319.4, 74.5)
- added U18: AD5254 - 50K, Package_SO:TSSOP-20_4.4x6.5mm_P0.65mm, F.Cu at (360.3, 61.8)
- added U19: AD5254 - 50K, Package_SO:TSSOP-20_4.4x6.5mm_P0.65mm, F.Cu at (369.1, 58.7)
- added U20: AD5254 - 50K, Package_SO:TSSOP-20_4.4x6.5mm_P0.65mm, F.Cu at (401.2, 40.2)
- added U21: AD5254 - 50K, Package_SO:TSSOP-20_4.4x6.5mm_P0.65mm, F.Cu at (377.8, 58.7)
- added U22: TCA9548APWR, Package_SO:TSSOP-24_4.4x7.8mm_P0.65mm, F.Cu at (351.6, 64.0)
- added U23: TPS92511DDA, Package_SO:SOIC-8-1EP_3.9x4.9mm_P1.27mm_EP2.29x3mm_ThermalVias, F.Cu at (361.5, 86.5)
- added U24: TPS92511DDA, Package_SO:SOIC-8-1EP_3.9x4.9mm_P1.27mm_EP2.29x3mm_ThermalVias, F.Cu at (361.4, 93.0)
- added U25: TPS92511DDA, Package_SO:SOIC-8-1EP_3.9x4.9mm_P1.27mm_EP2.29x3mm_ThermalVias, F.Cu at (394.9, 55.3)
- added U26: TPS92511DDA, Package_SO:SOIC-8-1EP_3.9x4.9mm_P1.27mm_EP2.29x3mm_ThermalVias, F.Cu at (370.2, 85.1)
- added U27: ADS1115IDGSR, Package_SO:MSOP-10_3x3mm_P0.5mm, F.Cu at (377.1, 65.1)
- added U28: TPS92511DDA, Package_SO:SOIC-8-1EP_3.9x4.9mm_P1.27mm_EP2.29x3mm_ThermalVias, F.Cu at (353.0, 91.2)
- added U29: TPS92511DDA, Package_SO:SOIC-8-1EP_3.9x4.9mm_P1.27mm_EP2.29x3mm_ThermalVias, F.Cu at (370.2, 78.7)
- added U30: TPS92511DDA, Package_SO:SOIC-8-1EP_3.9x4.9mm_P1.27mm_EP2.29x3mm_ThermalVias, F.Cu at (386.4, 62.6)
- added U31: TPS92511DDA, Package_SO:SOIC-8-1EP_3.9x4.9mm_P1.27mm_EP2.29x3mm_ThermalVias, F.Cu at (344.2, 97.2)
- added U6: TLV4314IPWR, Package_SO:TSSOP-14_4.4x5mm_P0.65mm, F.Cu at (310.7, 74.5)
- added U9: AD5242, Package_SO:TSSOP-16_4.4x5mm_P0.65mm, F.Cu at (367.5, 51.4)
- C14, C15, C16: value 10pF -> 0.1μF
- C19, C20, C21: value 0.1μF -> 10pF
- D10, D11, D14, D15, D16, D9: value B160-13-F -> 11-21/BHC-AQ2S1M/2T; footprint Diode_SMD:D_SMA -> LED_SMD:LED_1206_3216Metric
- D17, D18, D19, D20, D21, D24, D4, D5, D6, D8: value B160-13-F -> PMEG6010CEH; footprint Diode_SMD:D_SMA -> Diode_SMD:D_SOD-123F
- D22, D23: value 11-21/BHC-AQ2S1M/2T -> PMEG6010CEH; footprint LED_SMD:LED_1206_3216Metric -> Diode_SMD:D_SOD-123F
- L1, L2, L3, L4: value Pheonix 1841539 -> 680uH; footprint SamacSys_Parts:1841539 -> Inductor_SMD:L_6.3x6.3_H3
- Q2, Q3, Q4, Q5: value ULN2803ADWR -> DMN6140LQ-7; footprint Package_SO:SOIC-18W_7.5x11.6mm_P1.27mm -> Package_TO_SOT_SMD:SOT-23
- R1: value 33KΩ -> 330KΩ
- R19, R29, R30: value 33KΩ -> 10KΩ
- R20, R21, R24, R25: value 50Ω -> 10KΩ; footprint Resistor_SMD:R_2512_6332Metric -> Resistor_SMD:R_0402_1005Metric
- R22, R23, R26, R27: value 80Ω -> 10KΩ; footprint Resistor_SMD:R_0805_2012Metric -> Resistor_SMD:R_0402_1005Metric
- R4, R5, R6, R7: value 499KΩ -> 10KΩ
- U5: moved to F.Cu
- U7: value MCP23017-E/SO -> PCA9685PW; footprint Package_SO:SOIC-28W_7.5x17.9mm_P1.27mm -> Package_SO:TSSOP-28_4.4x9.7mm_P0.65mm
- U8: value MCP23017-E/SO -> AD5242; footprint Package_SO:SOIC-28W_7.5x17.9mm_P1.27mm -> Package_SO:TSSOP-16_4.4x5mm_P0.65mm
- moved Q11 336.5 mm to (430.4, 31.8)
- moved L4 336.1 mm to (418.4, 28.8)
- moved D23 331.4 mm to (416.9, 37.8)
- moved Q5 323.0 mm to (421.9, 38.4)
- moved D8 321.2 mm to (425.5, 26.6), turned to 0 degrees
- moved R26 320.0 mm to (426.6, 34.6), turned to 0 degrees
- moved R27 317.7 mm to (411.3, 54.1), turned to 0 degrees
- moved R25 317.3 mm to (418.0, 42.4), turned to 0 degrees
- moved D22 316.1 mm to (425.5, 29.9)
- moved C12 312.2 mm to (419.7, 56.1)
- moved C17 309.0 mm to (431.4, 47.0), turned to 0 degrees
- moved C4 306.1 mm to (427.0, 50.9)
- moved R24 302.2 mm to (418.0, 40.4), turned to 0 degrees
- moved L3 300.4 mm to (409.9, 36.7)
- moved R1 299.8 mm to (430.1, 43.0), turned to 0 degrees
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Connections:
- net /AIN1 renamed /AIN11
- C11 pad 1: +12V -> +5V
- C12 pad 1: +12V -> +5V
- C13 pad 1: /AVF1 -> /AVF11
- C13 pad 2: /PD1_NEG -> /PD11_NEG
- C14 pad 1: /AVF2 -> GND
- C14 pad 2: /PD2_NEG -> +5V
- C15 pad 1: /AVF3 -> GND
- C15 pad 2: /PD3_NEG -> +5V
- C16 pad 1: /AVF4 -> +5V
- C16 pad 2: /PD4_NEG -> GND
- C19 pad 1: GND -> /AVF12
- C19 pad 2: /AIN2 -> /PD12_NEG
- C20 pad 1: GND -> /AVF31
- C20 pad 2: /AIN3 -> /PD31_NEG
- C21 pad 1: GND -> /AVF32
- C21 pad 2: /AIN4 -> /PD32_NEG
- C5 pad 1: +5V -> GND
- C5 pad 2: GND -> +5V
- C8 pad 1: +12V -> GND
- C8 pad 2: GND -> +5V
- C9 pad 1: +12V -> GND
- C9 pad 2: GND -> +5V
- D10 pad 1: +12V -> Net-(D10-Pad1)
- D10 pad 2: /DAC1/A_WASTE2 -> +5V
- D11 pad 1: +12V -> Net-(D11-Pad1)
- D11 pad 2: /DAC1/FAN1_NEG -> +5V
- D14 pad 1: +12V -> Net-(D14-Pad1)
- D14 pad 2: /DAC2/A_DRUGS3 -> +5V
- D15 pad 1: +12V -> Net-(D15-Pad1)
- D15 pad 2: /DAC2/A_MEDIA3 -> +5V
- D16 pad 1: +12V -> Net-(D16-Pad1)
- D16 pad 2: /DAC2/A_WASTE3 -> +5V
- D17 pad 2: /DAC1/FAN2_NEG -> /DRUG21_NEG
- D18 pad 2: /DAC2/A_DRUGS4 -> /DRUG22_NEG
- D19 pad 2: /DAC2/A_MEDIA4 -> /MEDIA2_NEG
- D20 pad 2: /DAC2/A_WASTE4 -> /WASTE2_NEG
- D21 pad 2: /DAC2/FAN3_NEG -> /FAN2_NEG
- D22 pad 1: Net-(D22-Pad1) -> +12V
- D22 pad 2: +5V -> /DRUG31_NEG
- D23 pad 1: Net-(D23-Pad1) -> +12V
- D23 pad 2: +5V -> /DRUG32_NEG
- D24 pad 2: /DAC2/FAN4_NEG -> /MEDIA3_NEG
- D4 pad 2: /DAC1/A_DRUGS1 -> /DRUG12_NEG
- D5 pad 2: /DAC1/A_MEDIA1 -> /MEDIA1_NEG
- D6 pad 2: /DAC1/A_WASTE1 -> /WASTE1_NEG
- D8 pad 2: /DAC1/A_DRUGS2 -> /FAN1_NEG
- D9 pad 1: +12V -> Net-(D9-Pad1)
- D9 pad 2: /DAC1/A_MEDIA2 -> +5V
- L1 pad 1: /DAC1/A_DRUGS1 -> /LED11_CCNEG
- L1 pad 2: /DAC1/A_MEDIA1 -> /LED11_NEG
- L2 pad 1: /DAC1/A_DRUGS2 -> /LED31_CCNEG
- L2 pad 2: /DAC1/A_MEDIA2 -> /LED31_NEG
- L3 pad 1: /DAC2/A_DRUGS3 -> /LED12_CCNEG
- L3 pad 2: /DAC2/A_MEDIA3 -> /LED12_NEG
- L4 pad 1: /DAC2/A_DRUGS4 -> /LED32_CCNEG
- L4 pad 2: /DAC2/A_MEDIA4 -> /LED32_NEG
- Q10 pad 1: /FAN3_PWM -> /DRUGS11_PWM
- Q10 pad 3: /DAC2/FAN3_NEG -> (no net)
- Q11 pad 1: /FAN4_PWM -> /DRUGS21_PWM
- Q11 pad 3: /DAC2/FAN4_NEG -> (no net)
- Q2 pad 1: /DAC1/D_DRUGS1 -> /MEDIA1_PWM
- Q2 pad 2: /DAC1/D_MEDIA1 -> GND
- Q2 pad 3: /DAC1/D_WASTE1 -> /MEDIA1_NEG
- Q3 pad 1: /DAC1/D_DRUGS2 -> /MEDIA2_PWM
- Q3 pad 2: /DAC1/D_MEDIA2 -> GND
- Q3 pad 3: /DAC1/D_WASTE2 -> /MEDIA2_NEG
- Q4 pad 1: /DAC2/D_DRUGS3 -> /MEDIA3_PWM
- Q4 pad 2: /DAC2/D_MEDIA3 -> GND
- Q4 pad 3: /DAC2/D_WASTE3 -> /MEDIA3_NEG
- Q5 pad 1: /DAC2/D_DRUGS4 -> /MEDIA4_PWM
- Q5 pad 2: /DAC2/D_MEDIA4 -> GND
- Q5 pad 3: /DAC2/D_WASTE4 -> /MEDIA4_NEG
- Q8 pad 3: /DAC1/FAN1_NEG -> /FAN1_NEG
- Q9 pad 1: /FAN2_PWM -> /FAN3_PWM
- Q9 pad 3: /DAC1/FAN2_NEG -> /FAN3_NEG
- R1 pad 2: /ALP1 -> /ALP11
- R10 pad 2: /FAN2_PWM -> /FAN3_PWM
- R11 pad 2: /FAN3_PWM -> /DRUGS11_PWM
- R14 pad 2: /FAN4_PWM -> /DRUGS21_PWM
- R19 pad 1: /AIN2 -> +5V
- R19 pad 2: /ALP2 -> /DRUGS31_PWM
- R20 pad 1: /DAC1/A_LED1 -> +5V
- R20 pad 2: /DAC1/LED1_NEG -> /DRUGS41_PWM
- R21 pad 1: /DAC1/A_LED2 -> +5V
- R21 pad 2: /DAC1/LED2_NEG -> /FAN2_PWM
- R22 pad 1: /DAC1/A_IND1 -> +5V
- R22 pad 2: Net-(D12-Pad1) -> /FAN4_PWM
- R23 pad 1: /DAC1/A_IND2 -> Net-(R23-Pad1)
- R23 pad 2: Net-(D13-Pad1) -> GND
- R24 pad 1: /DAC2/A_LED3 -> +5V
- R24 pad 2: /DAC2/LED3_NEG -> /DRUGS12_PWM
- R25 pad 1: /DAC2/A_LED4 -> +5V
- R25 pad 2: /DAC2/LED4_NEG -> /DRUGS22_PWM
- R26 pad 1: /DAC2/A_IND3 -> +5V
- R26 pad 2: Net-(D22-Pad1) -> /DRUGS32_PWM
- R27 pad 1: /DAC2/A_IND4 -> +5V
- R27 pad 2: Net-(D23-Pad1) -> /DRUGS42_PWM
- R29 pad 1: /AIN3 -> Net-(R29-Pad1)
- R29 pad 2: /ALP3 -> GND
- R30 pad 1: /AIN4 -> +5V
- R30 pad 2: /ALP4 -> /WASTE1_PWM
- R32 pad 2: /V_REF -> /PD11_POS
- R4 pad 1: /AVF1 -> Net-(R4-Pad1)
- R4 pad 2: /PD1_NEG -> GND
- R5 pad 1: /AVF2 -> +5V
- R5 pad 2: /PD2_NEG -> /MEDIA1_PWM
- R6 pad 1: /AVF3 -> +5V
- R6 pad 2: /PD3_NEG -> /MEDIA2_PWM
- R7 pad 1: /AVF4 -> +5V
- R7 pad 2: /PD4_NEG -> /MEDIA3_PWM
- R8 pad 1: Net-(R8-Pad1) -> +5V
- R8 pad 2: GND -> /MEDIA4_PWM
- U1 pad 10: (no net) -> /LED11_PWM
- U1 pad 11: (no net) -> /LED12_PWM
- U1 pad 12: (no net) -> /IND11_PWM
- U1 pad 13: (no net) -> /IND12_PWM
- U1 pad 15: (no net) -> /MEDIA2_PWM
- U1 pad 16: (no net) -> /DRUGS21_PWM
- U1 pad 17: (no net) -> /DRUGS22_PWM
- U1 pad 18: (no net) -> /WASTE2_PWM
- U1 pad 19: (no net) -> /LED21_PWM
- U1 pad 20: (no net) -> /LED22_PWM
- U1 pad 21: (no net) -> /IND21_PWM
- U1 pad 22: (no net) -> /IND22_PWM
- U1 pad 25: Net-(R8-Pad1) -> Net-(R4-Pad1)
- U1 pad 26: /SCL -> /SCL-PWM
- U1 pad 27: /SDA -> /SDA-PWM
- U1 pad 5: +5V -> GND
- U1 pad 6: /FAN1_PWM -> /MEDIA1_PWM
- U1 pad 7: /FAN2_PWM -> /DRUGS11_PWM
- U1 pad 8: /FAN3_PWM -> /DRUGS12_PWM
- U1 pad 9: /FAN4_PWM -> /WASTE1_PWM
- U2 pad 10: /SCL -> /SCL-ADC
- U2 pad 5: /AIN2 -> /AIN12
- U2 pad 6: /AIN3 -> /AIN21
- U2 pad 7: /AIN4 -> /AIN22
- U2 pad 9: /SDA -> /SDA-ADC
- U3 pad 1: /AVF1 -> /AVF11
- U3 pad 10: /V_REF -> /PD11_POS
- U3 pad 12: /V_REF -> /PD11_POS
- U3 pad 13: /PD4_NEG -> /PD22_NEG
- U3 pad 14: /AVF4 -> /AVF22
- U3 pad 2: /PD1_NEG -> /PD11_NEG
- U3 pad 3: /V_REF -> /PD11_POS
- U3 pad 5: /V_REF -> /PD11_POS
- U3 pad 6: /PD2_NEG -> /PD12_NEG
- U3 pad 7: /AVF2 -> /AVF12
- U3 pad 8: /AVF3 -> /AVF21
- U3 pad 9: /PD3_NEG -> /PD21_NEG
- U4 pad 1: /ALP1 -> /ALP11
- U4 pad 10: /AVF3 -> /AVF21
- U4 pad 12: /AVF4 -> /AVF22
- U4 pad 13: /ALP4 -> /APOT11
- U4 pad 14: /ALP4 -> /ALP22
- U4 pad 2: /ALP1 -> /APOT11
- U4 pad 3: /AVF1 -> /AVF11
- U4 pad 5: /AVF2 -> /AVF12
- U4 pad 6: /ALP2 -> /APOT12
- U4 pad 7: /ALP2 -> /ALP12
- U4 pad 8: /ALP3 -> /ALP21
- U4 pad 9: /ALP3 -> /APOT11
- U5 pad 7: /V_REF -> /PD11_POS
- U5 pad 8: /V_REF -> /PD11_POS
- U7 pad 1: /DAC1/D_DRUGS2 -> +5V
- U7 pad 10: GND -> /LED31_PWM
- U7 pad 11: (no net) -> /LED32_PWM
- U7 pad 12: /SCL -> /IND31_PWM
- U7 pad 13: /SDA -> /IND32_PWM
- U7 pad 14: (no net) -> GND
- U7 pad 15: GND -> /MEDIA4_PWM
- U7 pad 16: GND -> /DRUGS41_PWM
- U7 pad 17: GND -> /DRUGS42_PWM
- U7 pad 18: +5V -> /WASTE4_PWM
- U7 pad 19: (no net) -> /LED41_PWM
- U7 pad 2: /DAC1/D_MEDIA2 -> GND
- U7 pad 20: (no net) -> /LED42_PWM
- U7 pad 21: /DAC1/D_DRUGS1 -> /IND41_PWM
- U7 pad 22: /DAC1/D_MEDIA1 -> /IND42_PWM
- U7 pad 23: /DAC1/D_WASTE1 -> GND
- U7 pad 24: /DAC1/D_LED1 -> GND
- U7 pad 25: /DAC1/D_IND1 -> Net-(R23-Pad1)
- U7 pad 26: (no net) -> /SCL-PWM
- U7 pad 27: (no net) -> /SDA-PWM
- U7 pad 28: (no net) -> +5V
- U7 pad 3: /DAC1/D_WASTE2 -> GND
- U7 pad 4: /DAC1/D_LED2 -> GND
- U7 pad 5: /DAC1/D_IND2 -> GND
- U7 pad 6: (no net) -> /MEDIA3_PWM
- U7 pad 7: (no net) -> /DRUGS31_PWM
- U7 pad 8: (no net) -> /DRUGS32_PWM
- U7 pad 9: +5V -> /WASTE3_PWM
- U8 pad 1: /DAC2/D_DRUGS4 -> (no net)
- U8 pad 11: (no net) -> GND
- U8 pad 12: /SCL -> GND
- U8 pad 13: /SDA -> (no net)
- U8 pad 14: (no net) -> /PD12_NEG
- U8 pad 15: +5V -> /AVF12
- U8 pad 16: GND -> (no net)
- U8 pad 2: /DAC2/D_MEDIA4 -> (no net)
- U8 pad 3: /DAC2/D_WASTE4 -> /AVF11
- U8 pad 4: /DAC2/D_LED4 -> /PD11_NEG
- U8 pad 5: /DAC2/D_IND4 -> +5V
- U8 pad 6: (no net) -> GND
- U8 pad 7: (no net) -> /SDA-1MPOT
- U8 pad 8: (no net) -> /SCL-1MPOT
- U8 pad 9: +5V -> GND
Routing:
- net /V_REF: track 214.7 -> 0.00 mm, vias 7 -> 0
- net /DAC1/A_DRUGS2: track 134.7 -> 0.00 mm, vias 2 -> 0
- net /DAC1/A_DRUGS1: track 125.7 -> 0.00 mm, vias 2 -> 0
- net /DAC1/A_MEDIA1: track 120.9 -> 0.00 mm, vias 2 -> 0
- net /DAC1/A_WASTE2: track 117.9 -> 0.00 mm, vias 2 -> 0
- net /DAC1/A_MEDIA2: track 116.4 -> 0.00 mm, vias 2 -> 0
- net /DAC1/A_WASTE1: track 111.6 -> 0.00 mm, vias 2 -> 0
- net +3V3: track 98.0 -> 1.60 mm, vias 4 -> 1
- net /PD1_NEG: track 96.0 -> 0.00 mm, vias 2 -> 0
- net /SDA: track 92.0 -> 0.00 mm, vias 5 -> 0
- net /DAC1/FAN1_NEG: track 83.4 -> 0.00 mm, vias 1 -> 0
- net /SCL: track 83.7 -> 0.29 mm, vias 5 -> 0
- net /PD2_NEG: track 82.8 -> 0.00 mm, vias 2 -> 0
- net /DAC2/A_WASTE3: track 81.5 -> 0.00 mm, vias 2 -> 0
- net GND: track 76.3 -> 0.00 mm, vias 15 -> 0
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- removed copper zone on In2.Cu, net +12V
- removed copper zone on In1.Cu, net +5V
- removed copper zone on B.Cu, net GND
- removed copper zone on F.Cu, net GND
Other:
- board outline removed
- board text removed: "+"
- board text removed: "-"
- board text removed: "CU1"
- board text removed: "CU2"
- board text removed: "CU3"
- board text removed: "CU4"
- board text removed: "DRUG"
- board text removed: "Designed by Vishhvaan"
- board text removed: "EVE_PCB"
- board text removed: "FAN"
- board text removed: "JLCJLCJLCJLC"
- board text removed: "LED"
- board text removed: "LOWER"
- board text removed: "MEDIA"
- board text removed: "PD"
- board text removed: "REV 4.82"
- board text removed: "UPPER"
- board text removed: "WASTE"

Commit message: Starting the wiring
Parts:
- removed J8, J9: Conn_01x18, ICs:282888-7
- J6: value Conn_01x18 -> Conn_02x18_Odd_Even; footprint ICs:282888-7 -> Connector_PinHeader_2.54mm:PinHeader_2x18_P2.54mm_Vertical
- J7: value Conn_01x18 -> Conn_02x22_Odd_Even; footprint ICs:282888-7 -> Connector_PinHeader_2.54mm:PinHeader_2x22_P2.54mm_Vertical
- moved Q21 321.7 mm to (106.7, 74.9)
- moved U20 310.8 mm to (91.4, 64.8)
- moved D8 303.2 mm to (127.0, 80.0)
- moved Q29 293.9 mm to (116.8, 74.9)
- moved D17 283.8 mm to (127.1, 85.1)
- moved Q25 280.5 mm to (111.8, 74.9)
- moved U8 279.5 mm to (73.7, 77.5)
- moved Q8 270.9 mm to (137.2, 68.6)
- moved Q2 270.0 mm to (111.8, 68.6)
- moved D5 266.4 mm to (127.1, 72.4)
- moved Q17 260.5 mm to (116.8, 68.6)
- moved Q10 256.7 mm to (106.7, 68.6)
- moved D6 255.8 mm to (127.0, 76.2)
- moved U4 254.7 mm to (73.7, 64.8)
- moved U2 254.5 mm to (82.5, 53.3)
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Connections:
- J6 pad 1: /MEDIA1_NEG -> +12V
- J6 pad 10: +12V -> /MEDIA2_NEG
- J6 pad 12: +12V -> /DRUG21_NEG
- J6 pad 14: /FAN1_POS -> /DRUG22_NEG
- J6 pad 15: +5V -> +12V
- J6 pad 16: +5V -> /WASTE2_NEG
- J6 pad 17: /PD11_POS -> +12V
- J6 pad 18: /PD11_POS -> /MEDIA3_NEG
- J6 pad 2: /DRUG11_NEG -> /MEDIA1_NEG
- J6 pad 3: /DRUG12_NEG -> +12V
- J6 pad 4: /WASTE1_NEG -> /DRUG11_NEG
- J6 pad 5: /FAN1_NEG -> +12V
- J6 pad 6: /LED11_NEG -> /DRUG12_NEG
- J6 pad 7: /LED12_NEG -> +12V
- J6 pad 8: /PD11_NEG -> /WASTE1_NEG
- J6 pad 9: /PD12_NEG -> +12V
- J7 pad 1: /MEDIA3_NEG -> /FAN1_POS
- J7 pad 10: +12V -> /PD12_NEG
- J7 pad 11: +12V -> /FAN2_POS
- J7 pad 12: +12V -> /FAN2_NEG
- J7 pad 13: +12V -> +5V
- J7 pad 14: /FAN3_POS -> /LED21_NEG
- J7 pad 16: +5V -> /LED22_NEG
- J7 pad 18: /PD11_POS -> /PD21_NEG
- J7 pad 2: /DRUG31_NEG -> /FAN1_NEG
- J7 pad 3: /DRUG32_NEG -> +5V
- J7 pad 4: /WASTE3_NEG -> /LED11_NEG
- J7 pad 5: /FAN3_NEG -> +5V
- J7 pad 6: /LED31_NEG -> /LED12_NEG
- J7 pad 7: /LED32_NEG -> /PD11_POS
- J7 pad 8: /PD31_NEG -> /PD11_NEG
- J7 pad 9: /PD32_NEG -> /PD11_POS

Commit message: Major placment updates
Parts:
- U10, U11, U15, U16, U18, U19, U5: moved to B.Cu
- U23, U24, U25, U26, U28, U29, U30, U31: footprint Package_SO:SOIC-8-1EP_3.9x4.9mm_P1.27mm_EP2.29x3mm_ThermalVias -> Package_SO:SOIC-8-1EP_3.9x4.9mm_P1.27mm_EP2.29x3mm
- moved Q22 341.6 mm to (101.6, 91.4)
- moved L5 341.2 mm to (65.0, 106.7), turned to 180 degrees
- moved L3 329.8 mm to (83.8, 86.4), turned to 180 degrees
- moved Q3 326.5 mm to (101.6, 85.1)
- moved Q11 324.0 mm to (109.2, 85.1)
- moved Q26 324.0 mm to (109.2, 91.4)
- moved Q30 321.4 mm to (117.1, 91.4)
- moved Q18 321.4 mm to (116.8, 85.1)
- moved D33 319.1 mm to (74.9, 85.1)
- moved U25 311.8 mm to (83.8, 77.5)
- moved U30 304.7 mm to (83.8, 97.8)
- moved D35 304.6 mm to (74.9, 105.4)
- moved L1 297.0 mm to (64.8, 86.4), turned to 180 degrees
- moved U23 296.9 mm to (64.8, 77.5)
- moved C35 293.9 mm to (118.6, 24.4), turned to 180 degrees
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Connections:
- Q10 pad 3: (no net) -> /DRUG11_NEG
- Q11 pad 3: (no net) -> /DRUG21_NEG
- Q13 pad 3: (no net) -> /DRUG31_NEG
- Q14 pad 3: (no net) -> /DRUG41_NEG
- Q17 pad 3: (no net) -> /DRUG12_NEG
- Q18 pad 3: (no net) -> /DRUG22_NEG
- Q19 pad 3: (no net) -> /DRUG32_NEG
- Q20 pad 3: (no net) -> /DRUG42_NEG
- U1 pad 16: /DRUGS21_PWM -> (no net)
- U1 pad 17: /DRUGS22_PWM -> (no net)
- U1 pad 7: /DRUGS11_PWM -> (no net)
- U1 pad 8: /DRUGS12_PWM -> (no net)
- U7 pad 16: /DRUGS41_PWM -> (no net)
- U7 pad 17: /DRUGS42_PWM -> (no net)
- U7 pad 7: /DRUGS31_PWM -> (no net)
- U7 pad 8: /DRUGS32_PWM -> (no net)
Routing:
- net +3V3: track 1.60 -> 270.5 mm, vias 1 -> 3
- net /SCL-3.3: track 0.00 -> 204.7 mm, vias 0 -> 2
- net /TEMP_DA-3.3: track 0.00 -> 197.1 mm, vias 0 -> 2
- net /SDA-3.3: track 0.00 -> 194.3 mm, vias 0 -> 2
- net /SCL-1MPOT: track 0.00 -> 182.0 mm, vias 0 -> 7
- net /SDA-1MPOT: track 0.00 -> 177.7 mm, vias 0 -> 5
- net /SCL-PWM: track 0.00 -> 101.7 mm, vias 0 -> 4
- net /SDA-PWM: track 0.00 -> 97.8 mm, vias 0 -> 4
- net /SCL: track 0.29 -> 71.2 mm, vias 0 -> 2
- net /SDA: track 0.00 -> 64.0 mm, vias 0 -> 2
- net /I2CM_A3: track 0.00 -> 35.4 mm
- net /I2CM_A2: track 0.00 -> 23.5 mm
- net /TEMP_DA: track 0.32 -> 20.7 mm
- net Net-(D7-Pad1): track 0.00 -> 19.5 mm
- net +5V: track 2.75 -> 19.6 mm, vias 1 -> 5
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- added copper zone on In2.Cu, net +12V
- added copper zone on In1.Cu, net +5V
- added copper zone on B.Cu, net GND
- added copper zone on F.Cu, net GND
Other:
- board outline added: 184.2 x 102.9 mm

Commit message: PCB updates
Parts:
- U12, U13, U8, U9: moved to B.Cu
- U23, U24, U25, U26, U28, U29, U30, U31: value TPS92511DDA -> TPS92511DDAR; footprint Package_SO:SOIC-8-1EP_3.9x4.9mm_P1.27mm_EP2.29x3mm -> Package_SO:HSOP-8-1EP_3.9x4.9mm_P1.27mm_EP2.41x3.1mm
- moved C43 274.4 mm to (30.2, 84.8)
- moved C48 257.0 mm to (42.9, 84.1)
- moved C46 242.2 mm to (30.0, 87.5)
- moved R73 228.3 mm to (47.3, 86.8)
- moved R2 226.9 mm to (75.2, 39.9)
- moved R68 226.2 mm to (41.4, 87.3)
- moved R70 215.0 mm to (48.4, 84.8)
- moved C2 210.8 mm to (83.3, 36.8)
- moved R31 208.9 mm to (75.2, 38.6), turned to 180 degrees
- moved C29 190.1 mm to (80.5, 80.5)
- moved C3 114.2 mm to (62.2, 95.4), turned to 0 degrees
- moved Q1 112.2 mm to (56.6, 90.9)
- moved R66 111.9 mm to (194.1, 40.1), turned to 180 degrees
- moved R32 111.9 mm to (155.2, 41.7), turned to 180 degrees
- moved C6 111.4 mm to (62.1, 92.9), turned to 0 degrees
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Connections:
- J6 pad 1: +12V -> /SDA-PWM
- J6 pad 10: /MEDIA2_NEG -> /DRUG12_NEG
- J6 pad 12: /DRUG21_NEG -> /WASTE1_NEG
- J6 pad 14: /DRUG22_NEG -> /MEDIA2_NEG
- J6 pad 16: /WASTE2_NEG -> /DRUG21_NEG
- J6 pad 18: /MEDIA3_NEG -> /DRUG22_NEG
- J6 pad 2: /MEDIA1_NEG -> /SCL-PWM
- J6 pad 20: /DRUG31_NEG -> /WASTE2_NEG
- J6 pad 22: /DRUG32_NEG -> /MEDIA3_NEG
- J6 pad 24: /WASTE3_NEG -> /DRUG31_NEG
- J6 pad 26: /MEDIA4_NEG -> /DRUG32_NEG
- J6 pad 28: /DRUG41_NEG -> /WASTE3_NEG
- J6 pad 3: +12V -> +5V
- J6 pad 30: /DRUG42_NEG -> /MEDIA4_NEG
- J6 pad 32: /WASTE4_NEG -> /DRUG41_NEG
- J6 pad 33: +5V -> +12V
- J6 pad 34: GND -> /DRUG42_NEG
- J6 pad 35: /SDA-PWM -> +12V
- J6 pad 36: /SCL-PWM -> /WASTE4_NEG
- J6 pad 4: /DRUG11_NEG -> GND
- J6 pad 6: /DRUG12_NEG -> /MEDIA1_NEG
- J6 pad 8: /WASTE1_NEG -> /DRUG11_NEG
- R58 pad 1: Net-(R58-Pad1) -> GND
- R58 pad 2: GND -> Net-(R58-Pad2)
- R59 pad 1: Net-(R59-Pad1) -> GND
- R59 pad 2: GND -> Net-(R59-Pad2)
- R68 pad 1: Net-(R68-Pad1) -> GND
- R68 pad 2: GND -> Net-(R68-Pad2)
- R69 pad 1: Net-(R69-Pad1) -> GND
- R69 pad 2: GND -> Net-(R69-Pad2)
- R70 pad 1: Net-(R70-Pad1) -> GND
- R70 pad 2: GND -> Net-(R70-Pad2)
- R71 pad 1: Net-(R71-Pad1) -> GND
- R71 pad 2: GND -> Net-(R71-Pad2)
- R73 pad 1: Net-(R73-Pad1) -> GND
- R73 pad 2: GND -> Net-(R73-Pad2)
- R74 pad 1: Net-(R74-Pad1) -> GND
- R74 pad 2: GND -> Net-(R74-Pad2)
- U18 pad 14: /SCL-POT -> /SCL-50KPOT
- U18 pad 9: /SDA-POT -> /SDA-50KPOT
- U19 pad 14: /SCL-POT -> /SCL-50KPOT
- U19 pad 9: /SDA-POT -> /SDA-50KPOT
- U20 pad 14: /SCL-POT -> /SCL-50KPOT
- U20 pad 9: /SDA-POT -> /SDA-50KPOT
- U21 pad 14: /SCL-POT -> /SCL-50KPOT
- U21 pad 9: /SDA-POT -> /SDA-50KPOT
- U22 pad 6: (no net) -> /SDA-50KPOT
- U22 pad 7: (no net) -> /SCL-50KPOT
- U23 pad 1: +5V -> Net-(C33-Pad2)
- U23 pad 5: Net-(C33-Pad2) -> Net-(R58-Pad2)
- U23 pad 6: /LED11_CCNEG -> /LED11_PWM
- U23 pad 7: /LED11_PWM -> /LED11_CCNEG
- U23 pad 8: Net-(R58-Pad1) -> +5V
- U24 pad 1: +5V -> Net-(C34-Pad2)
- U24 pad 5: Net-(C34-Pad2) -> Net-(R59-Pad2)
- U24 pad 6: /LED31_CCNEG -> /LED31_PWM
- U24 pad 7: /LED31_PWM -> /LED31_CCNEG
- U24 pad 8: Net-(R59-Pad1) -> +5V
- U25 pad 1: +5V -> Net-(C43-Pad2)
- U25 pad 5: Net-(C43-Pad2) -> Net-(R68-Pad2)
- U25 pad 6: /LED12_CCNEG -> /LED12_PWM
- U25 pad 7: /LED12_PWM -> /LED12_CCNEG
- U25 pad 8: Net-(R68-Pad1) -> +5V
- U26 pad 1: +5V -> Net-(C44-Pad2)
- U26 pad 5: Net-(C44-Pad2) -> Net-(R69-Pad2)
- U26 pad 6: /LED32_CCNEG -> /LED32_PWM
- U26 pad 7: /LED32_PWM -> /LED32_CCNEG
- U26 pad 8: Net-(R69-Pad1) -> +5V
- U28 pad 1: +5V -> Net-(C46-Pad2)
- U28 pad 5: Net-(C46-Pad2) -> Net-(R70-Pad2)
- U28 pad 6: /LED21_CCNEG -> /LED21_PWM
- U28 pad 7: /LED21_PWM -> /LED21_CCNEG
- U28 pad 8: Net-(R70-Pad1) -> +5V
- U29 pad 1: +5V -> Net-(C47-Pad2)
- U29 pad 5: Net-(C47-Pad2) -> Net-(R71-Pad2)
- U29 pad 6: /LED41_CCNEG -> /LED41_PWM
- U29 pad 7: /LED41_PWM -> /LED41_CCNEG
- U29 pad 8: Net-(R71-Pad1) -> +5V
- U30 pad 1: +5V -> Net-(C48-Pad2)
- U30 pad 5: Net-(C48-Pad2) -> Net-(R73-Pad2)
- U30 pad 6: /LED22_CCNEG -> /LED22_PWM
- U30 pad 7: /LED22_PWM -> /LED22_CCNEG
- U30 pad 8: Net-(R73-Pad1) -> +5V
- U31 pad 1: +5V -> Net-(C49-Pad2)
- U31 pad 5: Net-(C49-Pad2) -> Net-(R74-Pad2)
- U31 pad 6: /LED42_CCNEG -> /LED42_PWM
- U31 pad 7: /LED42_PWM -> /LED42_CCNEG
- U31 pad 8: Net-(R74-Pad1) -> +5V
- U6 pad 1: /AVF11 -> /AVF31
- U6 pad 14: /AVF22 -> /AVF42
- U6 pad 7: /AVF12 -> /AVF32
- U6 pad 8: /AVF21 -> /AVF41
Routing:
- net /PD11_POS: track 0.00 -> 360.4 mm, vias 0 -> 4
- net /SCL-50KPOT: track 0.00 -> 164.7 mm, vias 0 -> 3
- net /SDA-50KPOT: track 0.00 -> 155.5 mm, vias 0 -> 3
- net /SDA-ADC: track 0.00 -> 146.4 mm, vias 0 -> 5
- net /SCL-ADC: track 0.00 -> 146.1 mm, vias 0 -> 6
- net /LED42_PWM: track 0.00 -> 87.1 mm, vias 0 -> 4
- net +5V: track 19.6 -> 101.4 mm, vias 5 -> 31
- net /LED32_PWM: track 0.00 -> 75.8 mm, vias 0 -> 4
- net /WASTE4_NEG: track 0.00 -> 74.3 mm
- net /SDA-PWM: track 97.8 -> 162.7 mm
- net /SCL-PWM: track 101.7 -> 165.7 mm
- net /DRUG42_NEG: track 0.00 -> 61.0 mm
- net /LED41_PWM: track 0.00 -> 59.5 mm, vias 0 -> 2
- net /DRUG41_NEG: track 0.00 -> 56.9 mm
- net GND: track 6.38 -> 62.1 mm, vias 0 -> 12
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Other:
- board size 184.2 x 102.9 mm -> 184.2 x 81.5 mm
- net class 12v: trace_width 0.75 -> 0.45
- net class vref added: clearance 0.2, trace_width 0.5, via_dia 0.8, via_drill 0.4

Commit message: PCBv5 updates
Parts:
- moved C33 195.8 mm to (67.1, 61.6)
- moved C17 195.3 mm to (69.1, 43.1), turned to 180 degrees
- moved C8 192.2 mm to (63.1, 46.6)
- moved C18 190.1 mm to (74.7, 42.0)
- moved C13 189.3 mm to (72.9, 55.2), turned to 270 degrees
- moved R1 188.3 mm to (74.7, 43.3), turned to 180 degrees
- moved C4 186.0 mm to (73.9, 57.1)
- moved R58 184.8 mm to (72.8, 69.3)
- moved R64 181.8 mm to (77.7, 44.3), turned to 180 degrees
- moved C36 181.0 mm to (85.0, 41.9), turned to 180 degrees
- moved C39 179.8 mm to (77.7, 43.1)
- moved C19 176.9 mm to (74.4, 59.9), turned to 90 degrees
- moved C24 176.6 mm to (85.7, 58.9), turned to 90 degrees
- moved R61 174.6 mm to (85.0, 43.2)
- moved C31 170.3 mm to (92.3, 44.6)
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Connections:
- Q10 pad 1: /DRUGS11_PWM -> /DRUG11_PWM
- Q11 pad 1: /DRUGS21_PWM -> /DRUG21_PWM
- Q13 pad 1: /DRUGS31_PWM -> /DRUG31_PWM
- Q14 pad 1: /DRUGS41_PWM -> /DRUG41_PWM
- Q17 pad 1: /DRUGS12_PWM -> /DRUG12_PWM
- Q18 pad 1: /DRUGS22_PWM -> /DRUG22_PWM
- Q19 pad 1: /DRUGS32_PWM -> /DRUG32_PWM
- Q20 pad 1: /DRUGS42_PWM -> /DRUG42_PWM
- R11 pad 2: /DRUGS11_PWM -> /DRUG11_PWM
- R14 pad 2: /DRUGS21_PWM -> /DRUG21_PWM
- R19 pad 2: /DRUGS31_PWM -> /DRUG31_PWM
- R20 pad 2: /DRUGS41_PWM -> /DRUG41_PWM
- R24 pad 2: /DRUGS12_PWM -> /DRUG12_PWM
- R25 pad 2: /DRUGS22_PWM -> /DRUG22_PWM
- R26 pad 2: /DRUGS32_PWM -> /DRUG32_PWM
- R27 pad 2: /DRUGS42_PWM -> /DRUG42_PWM
- U1 pad 16: (no net) -> /DRUG21_PWM
- U1 pad 17: (no net) -> /DRUG22_PWM
- U1 pad 7: (no net) -> /DRUG11_PWM
- U1 pad 8: (no net) -> /DRUG12_PWM
- U20 pad 13: (no net) -> /APOT21
- U20 pad 19: (no net) -> /APOT22
- U4 pad 13: /APOT11 -> /APOT22
- U4 pad 9: /APOT11 -> /APOT21
- U7 pad 16: (no net) -> /DRUG41_PWM
- U7 pad 17: (no net) -> /DRUG42_PWM
- U7 pad 7: (no net) -> /DRUG31_PWM
- U7 pad 8: (no net) -> /DRUG32_PWM
Routing:
- net /PD31_NEG: track 18.0 -> 248.9 mm, vias 1 -> 2
- net /PD32_NEG: track 23.8 -> 253.5 mm, vias 1 -> 2
- net +5V: track 101.4 -> 329.2 mm, vias 31 -> 80
- net GND: track 62.1 -> 281.6 mm, vias 12 -> 63
- net /PD41_NEG: track 16.4 -> 218.5 mm, vias 3 -> 4
- net /PD42_NEG: track 25.3 -> 222.5 mm, vias 1 -> 2
- net /LED32_NEG: track 0.00 -> 150.7 mm, vias 0 -> 1
- net /WASTE2_NEG: track 0.00 -> 145.8 mm, vias 0 -> 2
- net /LED31_NEG: track 0.00 -> 131.9 mm, vias 0 -> 1
- net /MEDIA2_NEG: track 0.00 -> 126.7 mm, vias 0 -> 2
- net /FAN1_NEG: track 0.00 -> 123.6 mm, vias 0 -> 2
- net /DRUG21_NEG: track 0.00 -> 119.8 mm, vias 0 -> 2
- net /LED42_NEG: track 0.00 -> 118.7 mm, vias 0 -> 1
- net /DRUG22_NEG: track 0.00 -> 117.9 mm, vias 0 -> 2
- net /WASTE1_NEG: track 0.00 -> 116.6 mm, vias 0 -> 2
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Other:
- net class vref: clearance 0.2 -> 0.3
