File: Start Building/Circuit Board Files/EVE-PCB/v5/v5_proj/EVE-PCB-V4.sch (KiCad schematic (older format))
At the start: 148 parts, among them J1 PJ-102AH, J2 2x20 Male Header, J3 1725669, Q1 UA7805CKCT, Q12 DMN6140LQ-7, Q6 DMN6140LQ-7, Q7 DMN6140LQ-7, U2 ADS1115IDGSR, U3 TLV4314IPWR, U4 TLV4314IPWR, U5 MCP1501-10E/SN

Commit message: Finalize schematic
Parts:
- removed C14, C15, C16: 10pF, Capacitor_SMD:C_0402_1005Metric, symbol Device:C
- removed C19, C20, C21: 0.1μF, Capacitor_SMD:C_0402_1005Metric, symbol EVE-PCB-V4-rescue:C-Device-EVE-PCB-rescue
- removed D? (x4): B160-13-F, Diode_SMD:D_SMA, symbol EVE-PCB-V4-rescue:BAT43-Diode-EVE-PCB-rescue
- removed D?: 11-21/BHC-AQ2S1M/2T, LED_SMD:LED_1206_3216Metric, symbol Device:LED
- removed L? (x2): Pheonix 1841539, SamacSys_Parts:1841539, symbol EVE-PCB-V4-rescue:1841539-SamacSys_Parts
- removed Q? (x26): DMN6140LQ-7, Package_TO_SOT_SMD:SOT-23, symbol Transistor_FET:DMN10H220L
- removed R29, R30: 33KΩ, Resistor_SMD:R_0402_1005Metric, symbol EVE-PCB-V4-rescue:R-Device-EVE-PCB-rescue
- removed R4, R5: 499KΩ, Resistor_SMD:R_0402_1005Metric, symbol EVE-PCB-V4-rescue:R-Device-EVE-PCB-rescue
- removed R? (x2): 50Ω, Resistor_SMD:R_2512_6332Metric, symbol EVE-PCB-V4-rescue:R-Device-EVE-PCB-rescue
- removed R?: 80Ω, Resistor_SMD:R_0805_2012Metric, symbol Device:R
- removed R? (x26): 10KΩ, Resistor_SMD:R_0402_1005Metric, symbol EVE-PCB-V4-rescue:R-Device-EVE-PCB-rescue
- added C11, C12, C14, C15, C22, C23, C28, C29, C30, C31, C32, C36, C37, C38, C39, C40, C41, C42, C45, C5, C8, C9: 0.1μF, Capacitor_SMD:C_0402_1005Metric, symbol EVE-PCB-V4-rescue:C-Device-EVE-PCB-rescue
- added C19, C20, C21, C24, C25, C26, C27: 10pF, Capacitor_SMD:C_0402_1005Metric, symbol Device:C
- added C33, C34, C43, C44, C46, C47, C48, C49: 2.2μF, Capacitor_SMD:C_0603_1608Metric, symbol EVE-PCB-V4-rescue:C-Device-EVE-PCB-rescue
- added D10, D11, D12, D13, D14, D15, D16: 11-21/BHC-AQ2S1M/2T, LED_SMD:LED_1206_3216Metric, symbol Device:LED
- added D17, D18, D19, D20, D21, D22, D23, D24, D25, D26, D27, D28, D29, D30, D31, D32, D33, D34, D35, D36, D37, D38, D39, D4: PMEG6010CEH, Diode_SMD:D_SOD-123F, symbol EVE-PCB-V4-rescue:BAT43-Diode-EVE-PCB-rescue
- added J5: Conn_02x03_Odd_Even, Connector_PinHeader_2.54mm:PinHeader_2x03_P2.54mm_Vertical, symbol Connector_Generic:Conn_02x03_Odd_Even
- added J6, J7, J8, J9: Conn_01x18, ICs:282888-7, symbol Connector_Generic:Conn_01x18
- added L1, L2, L3, L4, L5, L6, L7, L8: 680uH, Inductor_SMD:L_6.3x6.3_H3, symbol Device:L
- added Q11, Q13, Q14, Q18, Q19, Q20, Q22, Q23, Q24, Q26, Q27, Q28, Q3, Q30, Q31, Q32, Q4, Q5: DMN6140LQ-7, Package_TO_SOT_SMD:SOT-23, symbol Transistor_FET:DMN10H220L
- added R14, R20, R25, R26, R27, R33, R34, R35, R39, R40, R41, R43, R44, R45, R57, R60, R72, R8: 10KΩ, Resistor_SMD:R_0402_1005Metric, symbol EVE-PCB-V4-rescue:R-Device-EVE-PCB-rescue
- added R36, R37, R46, R47: 0.4Ω, Resistor_SMD:R_2512_6332Metric, symbol EVE-PCB-V4-rescue:R-Device-EVE-PCB-rescue
- added R49, R50, R51, R52, R53, R54, R55: 80Ω, Resistor_SMD:R_0805_2012Metric, symbol Device:R
- added R58, R59, R68, R69, R70, R71, R73, R74: 20KΩ, Resistor_SMD:R_0402_1005Metric, symbol EVE-PCB-V4-rescue:R-Device-EVE-PCB-rescue
- added R61, R62, R63, R64, R65, R66, R67: 330KΩ, Resistor_SMD:R_0402_1005Metric, symbol EVE-PCB-V4-rescue:R-Device-EVE-PCB-rescue
- added U10, U11, U15, U16: INA219AxDCN, Package_TO_SOT_SMD:SOT-23-8, symbol Analog_ADC:INA219AxDCN
- added U12, U13, U8, U9: AD5242, Package_SO:TSSOP-16_4.4x5mm_P0.65mm, symbol Potentiometer_Digital:AD5282
- added U17, U6: TLV4314IPWR, Package_SO:TSSOP-14_4.4x5mm_P0.65mm, symbol EVE-PCB-V4-rescue:LM324DR-LM324DR
- added U18, U19, U20, U21: AD5254 - 50K, Package_SO:TSSOP-20_4.4x6.5mm_P0.65mm, symbol Potentiometer_Digital:AD5254
- added U23, U24, U25, U26, U28, U29, U30, U31: TPS92511DDA, Package_SO:SOIC-8-1EP_3.9x4.9mm_P1.27mm_EP2.29x3mm_ThermalVias, symbol TPS92511DDA:TPS92511DDA
- added U27: ADS1115IDGSR, Package_SO:MSOP-10_3x3mm_P0.5mm, symbol EVE-PCB-V4-rescue:ADS1015IDGSR-ADS1015IDGSR
- D2, D5, D6, D8: renamed from D?; value B160-13-F -> PMEG6010CEH; footprint Diode_SMD:D_SMA -> Diode_SMD:D_SOD-123F; LCSC C24784 -> C110797
- R1: value 33KΩ -> 330KΩ; LCSC C25779 -> C25778
- R19: value 33KΩ -> 10KΩ; LCSC C25779 -> C25744
- R6, R7: value 499KΩ -> 10KΩ; LCSC C25793 -> C25744; Power 25E-6 -> low
- gave numbers to parts that had none: 35
Connections:
- net labels added: AIN11, AIN12, AIN21, AIN22, AIN31, AIN32, AIN41, AIN42, ALP11, ALP12, ALP21, ALP22, ALP31, ALP32, ALP41, ALP42, APOT11, APOT12, APOT21, APOT22, APOT31, APOT32, APOT41, APOT42, AVF11, AVF12, AVF21, AVF22, AVF31, AVF32, AVF41, AVF42, DRUG11_NEG, DRUG11_POS, DRUG12_NEG, DRUG12_POS, DRUG21_NEG, DRUG21_POS, DRUG22_NEG, DRUG22_POS, DRUG31_NEG, DRUG31_POS, DRUG32_NEG, DRUG32_POS, DRUG41_NEG, DRUG41_POS, DRUG42_NEG, DRUG42_POS, DRUGS21_NEG, DRUGS22_NEG, DRUGS31_NEG, DRUGS32_NEG, DRUGS41_NEG, DRUGS42_NEG, FAN1_POSS, FAN2_POSS, FAN3_POS, FAN3_POSS, FAN4_POS, FAN4_POSS, I2CM_A1, I2CM_A2, I2CM_A3, IND11_POS, IND12_POS, IND21_NEG, IND21_POS, IND22_NEG, IND22_POS, IND31_NEG, IND31_POS, IND32_NEG, IND32_POS, IND41_NEG, IND41_POS, IND42_NEG, IND42_POS, LED11_CCNEG, LED11_POS, LED11_SVIN, LED12_CCNEG, LED12_POS, LED12_SVIN, LED21_CCNEG, LED21_NEG, LED21_POS, LED21_SVIN, LED22_CCNEG, LED22_NEG, LED22_POS, LED22_SVIN, LED31_CCNEG, LED31_NEG, LED31_POS, LED31_SVIN, LED32_CCNEG, LED32_NEG, LED32_POS, LED32_SVIN, LED41_CCNEG, LED41_NEG, LED41_POS, LED41_SVIN, LED42_CCNEG, LED42_NEG, LED42_POS, LED42_SVIN, MEDIA3_NEG, MEDIA3_POS, MEDIA4_NEG, MEDIA4_POS, PD11_NEG, PD11_POS, PD12_NEG, PD12_POS, PD21_NEG, PD21_POS, PD22_NEG, PD22_POS, PD31_NEG, PD31_POS, PD32_NEG, PD32_POS, PD41_NEG, PD41_POS, PD42_NEG, PD42_POS, SCL-10KPOT, SCL-1MPOT, SCL-ADC, SCL-CUR, SCL-POT, SDA-10KPOT, SDA-1MPOT, SDA-ADC, SDA-CUR, SDA-POT, WASTE3_NEG, WASTE3_POS, WASTE4_NEG, WASTE4_POS
- net labels removed: AIN1, AIN2, AIN3, AIN4, ALP1, ALP2, ALP3, ALP4, AVF1, AVF2, AVF3, AVF4, A_IND1, A_IND2, A_LED1, A_LED2, DRUG1_NEG, DRUG1_POS, DRUG2_NEG, DRUG2_POS, IND1_POS, IND2_POS, LED1_NEG, LED1_POS, LED2_NEG, LED2_POS, PD1_NEG, PD1_POS, PD2_NEG, PD2_POS, PD3_NEG, PD4_NEG
- wire segments 663 -> 1277
- no-connect marks 66 -> 90
Other:
- moved on the sheet: C10, C13, C16, C17, C18, C2, C35, C4, C7, D2, D3, D5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

Commit message: Starting the wiring
Parts:
- removed J6, J7, J8, J9: Conn_01x18, ICs:282888-7, symbol Connector_Generic:Conn_01x18
- added J6: Conn_02x18_Odd_Even, Connector_PinHeader_2.54mm:PinHeader_2x18_P2.54mm_Vertical, symbol Connector_Generic:Conn_02x18_Odd_Even
- added J7: Conn_02x22_Odd_Even, Connector_PinHeader_2.54mm:PinHeader_2x22_P2.54mm_Vertical, symbol Connector_Generic:Conn_02x22_Odd_Even
Connections:
- wire segments 1277 -> 1289

Commit message: Major placment updates
Parts:
- U23, U24, U25, U26, U28, U29, U30, U31: footprint Package_SO:SOIC-8-1EP_3.9x4.9mm_P1.27mm_EP2.29x3mm_ThermalVias -> Package_SO:SOIC-8-1EP_3.9x4.9mm_P1.27mm_EP2.29x3mm
Connections:
- net DRUGS11_NEG is gone; now on net DRUG11_NEG: Q10.3 (D)
- net DRUGS12_NEG is gone; now on net DRUG12_NEG: Q17.3 (D)
- net DRUGS21_NEG is gone; now on net DRUG21_NEG: Q11.3 (D)
- net DRUGS22_NEG is gone; now on net DRUG22_NEG: Q18.3 (D)
- net DRUGS31_NEG is gone; now on net DRUG31_NEG: Q13.3 (D)
- net DRUGS32_NEG is gone; now on net DRUG32_NEG: Q19.3 (D)
- net DRUGS41_NEG is gone; now on net DRUG41_NEG: Q14.3 (D)
- net DRUGS42_NEG is gone; now on net DRUG42_NEG: Q20.3 (D)
- net DRUGS11_PWM: no longer U1.7 (LED1)
- net DRUGS12_PWM: no longer U1.8 (LED2)
- net DRUGS21_PWM: no longer U1.16 (LED9)
- net DRUGS22_PWM: no longer U1.17 (LED10)
- net DRUGS31_PWM: no longer U7.7 (LED1)
- net DRUGS32_PWM: no longer U7.8 (LED2)
- net DRUGS41_PWM: no longer U7.16 (LED9)
- net DRUGS42_PWM: no longer U7.17 (LED10)
- new net DRUG11_PWM: U1.7 (LED1)
- new net DRUG12_PWM: U1.8 (LED2)
- new net DRUG21_PWM: U1.16 (LED9)
- new net DRUG22_PWM: U1.17 (LED10)
- new net DRUG31_PWM: U7.7 (LED1)
- new net DRUG32_PWM: U7.8 (LED2)
- new net DRUG41_PWM: U7.16 (LED9)
- new net DRUG42_PWM: U7.17 (LED10)
Changed lines of the file:
@@
 MEDIA1_PWM
 Text Label 3350 11100 2    50   ~ 0
-DRUGS11_PWM
+DRUG11_PWM
 Text Label 3350 11200 2    50   ~ 0
-DRUGS12_PWM
+DRUG12_PWM
 Text Label 3350 11300 2    50   ~ 0
 WASTE1_PWM
@@
 MEDIA2_PWM
 Text Label 3350 11900 2    50   ~ 0
-DRUGS21_PWM
+DRUG21_PWM
 Text Label 3350 12000 2    50   ~ 0
-DRUGS22_PWM
+DRUG22_PWM
 Text Label 3350 12100 2    50   ~ 0
 WASTE2_PWM
@@
 MEDIA3_PWM
 Text Label 6100 11100 2    50   ~ 0
-DRUGS31_PWM
+DRUG31_PWM
 Text Label 6100 11200 2    50   ~ 0
-DRUGS32_PWM
+DRUG32_PWM
 Text Label 6100 11300 2    50   ~ 0
 WASTE3_PWM
@@
 MEDIA4_PWM
 Text Label 6100 11900 2    50   ~ 0
-DRUGS41_PWM
+DRUG41_PWM
 Text Label 6100 12000 2    50   ~ 0
-DRUGS42_PWM
+DRUG42_PWM
 Text Label 6100 12100 2    50   ~ 0
 WASTE4_PWM
@@
 	2100 13500 2100 13750
 Text Label 4400 13500 2    50   ~ 0
-DRUGS11_NEG
+DRUG11_NEG
 Wire Wire Line
 	4400 13500 3900 13500
@@
 	3900 13500 3900 13750
 Text Label 6250 13500 2    50   ~ 0
-DRUGS12_NEG
+DRUG12_NEG
 Wire Wire Line
 	6250 13500 5750 13500
@@
 	2100 14950 2100 15200
 Text Label 4400 14950 2    50   ~ 0
-DRUGS21_NEG
+DRUG21_NEG
 Wire Wire Line
 	4400 14950 3900 14950
@@
 	3900 14950 3900 15200
 Text Label 6250 14950 2    50   ~ 0
-DRUGS22_NEG
+DRUG22_NEG
 Wire Wire Line
 	6250 14950 5750 14950
@@
 	2100 16450 2100 16700
 Text Label 4400 16450 2    50   ~ 0
-DRUGS31_NEG
+DRUG31_NEG
 Wire Wire Line
 	4400 16450 3900 16450
@@
 	3900 16450 3900 16700
 Text Label 6250 16450 2    50   ~ 0
-DRUGS32_NEG
+DRUG32_NEG
 Wire Wire Line
 	6250 16450 5750 16450
@@
 	2100 18100 2100 18350
 Text Label 4400 18100 2    50   ~ 0
-DRUGS41_NEG
+DRUG41_NEG
 Wire Wire Line
 	4400 18100 3900 18100
@@
 	3900 18100 3900 18350
 Text Label 6250 18100 2    50   ~ 0
-DRUGS42_NEG
+DRUG42_NEG
 Wire Wire Line
 	6250 18100 5750 18100
@@
 F 0 "U23" H 19200 15570 50  0000 C CNN
 F 1 "TPS92511DDA" H 19200 15479 50  0000 C CNN
-F 2 "Package_SO:SOIC-8-1EP_3.9x4.9mm_P1.27mm_EP2.29x3mm_ThermalVias" H 19200 14600 50  0001 L BNN
+F 2 "Package_SO:SOIC-8-1EP_3.9x4.9mm_P1.27mm_EP2.29x3mm" H 19200 14600 50  0001 L BNN
 F 3 "" H 19200 14600 50  0001 C CNN
 F 4 "C114277" H 19200 14600 50  0001 C CNN "LCSC"
@@
 F 0 "U25" H 22550 15570 50  0000 C CNN
 F 1 "TPS92511DDA" H 22550 15479 50  0000 C CNN
-F 2 "Package_SO:SOIC-8-1EP_3.9x4.9mm_P1.27mm_EP2.29x3mm_ThermalVias" H 22550 14600 50  0001 L BNN
+F 2 "Package_SO:SOIC-8-1EP_3.9x4.9mm_P1.27mm_EP2.29x3mm" H 22550 14600 50  0001 L BNN
 F 3 "" H 22550 14600 50  0001 C CNN
 F 4 "C114277" H 22550 14600 50  0001 C CNN "LCSC"
@@
 F 0 "U28" H 25850 15570 50  0000 C CNN
 F 1 "TPS92511DDA" H 25850 15479 50  0000 C CNN
-F 2 "Package_SO:SOIC-8-1EP_3.9x4.9mm_P1.27mm_EP2.29x3mm_ThermalVias" H 25850 14600 50  0001 L BNN
+F 2 "Package_SO:SOIC-8-1EP_3.9x4.9mm_P1.27mm_EP2.29x3mm" H 25850 14600 50  0001 L BNN
 F 3 "" H 25850 14600 50  0001 C CNN
 F 4 "C114277" H 25850 14600 50  0001 C CNN "LCSC"
@@
 F 0 "U30" H 29300 15570 50  0000 C CNN
 F 1 "TPS92511DDA" H 29300 15479 50  0000 C CNN
-F 2 "Package_SO:SOIC-8-1EP_3.9x4.9mm_P1.27mm_EP2.29x3mm_ThermalVias" H 29300 14600 50  0001 L BNN
+F 2 "Package_SO:SOIC-8-1EP_3.9x4.9mm_P1.27mm_EP2.29x3mm" H 29300 14600 50  0001 L BNN
 F 3 "" H 29300 14600 50  0001 C CNN
 F 4 "C114277" H 29300 14600 50  0001 C CNN "LCSC"
@@
 F 0 "U24" H 19200 18670 50  0000 C CNN
 F 1 "TPS92511DDA" H 19200 18579 50  0000 C CNN
-F 2 "Package_SO:SOIC-8-1EP_3.9x4.9mm_P1.27mm_EP2.29x3mm_ThermalVias" H 19200 17700 50  0001 L BNN
+F 2 "Package_SO:SOIC-8-1EP_3.9x4.9mm_P1.27mm_EP2.29x3mm" H 19200 17700 50  0001 L BNN
 F 3 "" H 19200 17700 50  0001 C CNN
 F 4 "C114277" H 19200 17700 50  0001 C CNN "LCSC"
@@
 F 0 "U26" H 22550 18670 50  0000 C CNN
 F 1 "TPS92511DDA" H 22550 18579 50  0000 C CNN
-F 2 "Package_SO:SOIC-8-1EP_3.9x4.9mm_P1.27mm_EP2.29x3mm_ThermalVias" H 22550 17700 50  0001 L BNN
+F 2 "Package_SO:SOIC-8-1EP_3.9x4.9mm_P1.27mm_EP2.29x3mm" H 22550 17700 50  0001 L BNN
 F 3 "" H 22550 17700 50  0001 C CNN
 F 4 "C114277" H 22550 17700 50  0001 C CNN "LCSC"
@@
 F 0 "U29" H 25850 18670 50  0000 C CNN
 F 1 "TPS92511DDA" H 25850 18579 50  0000 C CNN
-F 2 "Package_SO:SOIC-8-1EP_3.9x4.9mm_P1.27mm_EP2.29x3mm_ThermalVias" H 25850 17700 50  0001 L BNN
+F 2 "Package_SO:SOIC-8-1EP_3.9x4.9mm_P1.27mm_EP2.29x3mm" H 25850 17700 50  0001 L BNN
 F 3 "" H 25850 17700 50  0001 C CNN
 F 4 "C114277" H 25850 17700 50  0001 C CNN "LCSC"
@@
 F 0 "U31" H 29300 18670 50  0000 C CNN
 F 1 "TPS92511DDA" H 29300 18579 50  0000 C CNN
-F 2 "Package_SO:SOIC-8-1EP_3.9x4.9mm_P1.27mm_EP2.29x3mm_ThermalVias" H 29300 17700 50  0001 L BNN
+F 2 "Package_SO:SOIC-8-1EP_3.9x4.9mm_P1.27mm_EP2.29x3mm" H 29300 17700 50  0001 L BNN
 F 3 "" H 29300 17700 50  0001 C CNN
 F 4 "C114277" H 29300 17700 50  0001 C CNN "LCSC"

Commit message: PCB updates
Parts:
- removed U23, U24, U25, U26, U28, U29, U30, U31: TPS92511DDA, Package_SO:SOIC-8-1EP_3.9x4.9mm_P1.27mm_EP2.29x3mm, symbol TPS92511DDA:TPS92511DDA
- added U23, U24, U25, U26, U28, U29, U30, U31: TPS92511DDAR, Package_SO:HSOP-8-1EP_3.9x4.9mm_P1.27mm_EP2.41x3.1mm, symbol TPS92511DDA:TPS92511DDAR
Connections:
- net SCL-POT is gone; now on net SCL-50KPOT: U18.14 (SCL), U19.14 (SCL), U20.14 (SCL), U21.14 (SCL)
- net SDA-POT is gone; now on net SDA-50KPOT: U18.9 (SDA), U19.9 (SDA), U20.9 (SDA), U21.9 (SDA)
- net +12V: now also J6.33 (Pin_33), J6.35 (Pin_35); no longer J6.1 (Pin_1), J6.3 (Pin_3)
- net +5V: now also J6.3 (Pin_3), U23.8 (VIN), U24.8 (VIN), U25.8 (VIN), U26.8 (VIN), U28.8 (VIN), U29.8 (VIN), U30.8 (VIN), U31.8 (VIN); no longer J6.33 (Pin_33)
- net AVF11: no longer U6.1 (1OUT)
- net AVF12: no longer U6.7 (2OUT)
- net AVF21: no longer U6.8 (3OUT)
- net AVF22: no longer U6.14 (4OUT)
- net AVF31: now also U6.1 (1OUT)
- net AVF32: now also U6.7 (2OUT)
- net AVF41: now also U6.8 (3OUT)
- net AVF42: now also U6.14 (4OUT)
- net DRUG11_NEG: now also J6.8 (Pin_8); no longer J6.4 (Pin_4)
- net DRUG12_NEG: now also J6.10 (Pin_10); no longer J6.6 (Pin_6)
- net DRUG21_NEG: now also J6.16 (Pin_16); no longer J6.12 (Pin_12)
- net DRUG22_NEG: now also J6.18 (Pin_18); no longer J6.14 (Pin_14)
- net DRUG31_NEG: now also J6.24 (Pin_24); no longer J6.20 (Pin_20)
- net DRUG32_NEG: now also J6.26 (Pin_26); no longer J6.22 (Pin_22)
- net DRUG41_NEG: now also J6.32 (Pin_32); no longer J6.28 (Pin_28)
- net DRUG42_NEG: now also J6.34 (Pin_34); no longer J6.30 (Pin_30)
- net GND: now also J6.4 (Pin_4), R58.1, R59.1, R68.1, R69.1, R70.1, R71.1, R73.1, R74.1, U23.2 (PGND), U23.4 (GND), U24.2 (PGND), U24.4 (GND), U25.2 (PGND), U25.4 (GND), U26.2 (PGND), U26.4 (GND), U28.2 (PGND), U28.4 (GND), U29.2 (PGND), U29.4 (GND), U30.2 (PGND), U30.4 (GND), U31.2 (PGND), U31.4 (GND); no longer J6.34 (Pin_34), R58.2, R59.2, R68.2, R69.2, R70.2, R71.2, R73.2, R74.2
- net LED11_CCNEG: now also U23.7 (LX)
- net LED11_PWM: now also U23.6 (DIM)
- net LED11_SVIN: now also U23.3 (IADJ)
- net LED12_CCNEG: now also U25.7 (LX)
- net LED12_PWM: now also U25.6 (DIM)
- net LED12_SVIN: now also U25.3 (IADJ)
- net LED21_CCNEG: now also U28.7 (LX)
- net LED21_PWM: now also U28.6 (DIM)
- net LED21_SVIN: now also U28.3 (IADJ)
- net LED22_CCNEG: now also U30.7 (LX)
- net LED22_PWM: now also U30.6 (DIM)
- net LED22_SVIN: now also U30.3 (IADJ)
- net LED31_CCNEG: now also U24.7 (LX)
- net LED31_PWM: now also U24.6 (DIM)
- net LED31_SVIN: now also U24.3 (IADJ)
- net LED32_CCNEG: now also U26.7 (LX)
- net LED32_PWM: now also U26.6 (DIM)
- net LED32_SVIN: now also U26.3 (IADJ)
- net LED41_CCNEG: now also U29.7 (LX)
- net LED41_PWM: now also U29.6 (DIM)
- net LED41_SVIN: now also U29.3 (IADJ)
- net LED42_CCNEG: now also U31.7 (LX)
- net LED42_PWM: now also U31.6 (DIM)
- net LED42_SVIN: now also U31.3 (IADJ)
- net MEDIA1_NEG: now also J6.6 (Pin_6); no longer J6.2 (Pin_2)
- net MEDIA2_NEG: now also J6.14 (Pin_14); no longer J6.10 (Pin_10)
- net MEDIA3_NEG: now also J6.22 (Pin_22); no longer J6.18 (Pin_18)
- net MEDIA4_NEG: now also J6.30 (Pin_30); no longer J6.26 (Pin_26)
- net SCL-PWM: now also J6.2 (Pin_2); no longer J6.36 (Pin_36)
- net SDA-PWM: now also J6.1 (Pin_1); no longer J6.35 (Pin_35)
- net WASTE1_NEG: now also J6.12 (Pin_12); no longer J6.8 (Pin_8)
- net WASTE2_NEG: now also J6.20 (Pin_20); no longer J6.16 (Pin_16)
- net WASTE3_NEG: now also J6.28 (Pin_28); no longer J6.24 (Pin_24)
- net WASTE4_NEG: now also J6.36 (Pin_36); no longer J6.32 (Pin_32)
- net at C33.2: now also U23.1 (VCC)
- net at C43.2: now also U25.1 (VCC)
- net at C46.2: now also U28.1 (VCC)
- net at C48.2: now also U30.1 (VCC)
- net at C34.2: now also U24.1 (VCC)
- net at C44.2: now also U26.1 (VCC)
- net at C47.2: now also U29.1 (VCC)
- net at C49.2: now also U31.1 (VCC)
- net SCL-10KPOT renamed SCL-50KPOT
- net SDA-10KPOT renamed SDA-50KPOT
- new net: R58.2, U23.5 (FS)
- new net: R68.2, U25.5 (FS)
- new net: R70.2, U28.5 (FS)
- new net: R73.2, U30.5 (FS)
- new net: R59.2, U24.5 (FS)
- new net: R69.2, U26.5 (FS)
- new net: R71.2, U29.5 (FS)
- new net: R74.2, U31.5 (FS)
- no-connect marks 90 -> 98
Other:
- moved on the sheet: C33, R58

Commit message: PCBv5 updates
Connections:
- net DRUGS11_PWM is gone; now on net DRUG11_PWM: Q10.1 (G), R11.2
- net DRUGS12_PWM is gone; now on net DRUG12_PWM: Q17.1 (G), R24.2
- net DRUGS21_PWM is gone; now on net DRUG21_PWM: Q11.1 (G), R14.2
- net DRUGS22_PWM is gone; now on net DRUG22_PWM: Q18.1 (G), R25.2
- net DRUGS31_PWM is gone; now on net DRUG31_PWM: Q13.1 (G), R19.2
- net DRUGS32_PWM is gone; now on net DRUG32_PWM: Q19.1 (G), R26.2
- net DRUGS41_PWM is gone; now on net DRUG41_PWM: Q14.1 (G), R20.2
- net DRUGS42_PWM is gone; now on net DRUG42_PWM: Q20.1 (G), R27.2
- net APOT11: no longer U4.13 (4IN-), U4.9 (3IN-)
- net APOT21: now also U4.9 (3IN-)
- net APOT22: now also U4.13 (4IN-)
Changed lines of the file:
@@
 $EndComp
 Text Label 2600 13950 0    50   ~ 0
-DRUGS11_PWM
+DRUG11_PWM
 $Comp
 L EVE-PCB-V4-rescue:+5V-power-EVE-PCB-rescue #PWR0137
@@
 $EndComp
 Text Label 4500 13950 0    50   ~ 0
-DRUGS12_PWM
+DRUG12_PWM
 $Comp
 L EVE-PCB-V4-rescue:+5V-power-EVE-PCB-rescue #PWR0139
@@
 $EndComp
 Text Label 2600 15400 0    50   ~ 0
-DRUGS21_PWM
+DRUG21_PWM
 $Comp
 L EVE-PCB-V4-rescue:+5V-power-EVE-PCB-rescue #PWR0145
@@
 $EndComp
 Text Label 4500 15400 0    50   ~ 0
-DRUGS22_PWM
+DRUG22_PWM
 $Comp
 L EVE-PCB-V4-rescue:+5V-power-EVE-PCB-rescue #PWR0147
@@
 $EndComp
 Text Label 2600 16900 0    50   ~ 0
-DRUGS31_PWM
+DRUG31_PWM
 $Comp
 L EVE-PCB-V4-rescue:+5V-power-EVE-PCB-rescue #PWR0153
@@
 $EndComp
 Text Label 4500 16900 0    50   ~ 0
-DRUGS32_PWM
+DRUG32_PWM
 $Comp
 L EVE-PCB-V4-rescue:+5V-power-EVE-PCB-rescue #PWR0155
@@
 $EndComp
 Text Label 2600 18550 0    50   ~ 0
-DRUGS41_PWM
+DRUG41_PWM
 $Comp
 L EVE-PCB-V4-rescue:+5V-power-EVE-PCB-rescue #PWR0161
@@
 $EndComp
 Text Label 4500 18550 0    50   ~ 0
-DRUGS42_PWM
+DRUG42_PWM
 $Comp
 L EVE-PCB-V4-rescue:+5V-power-EVE-PCB-rescue #PWR0163
@@
 APOT12
 Text Label 13100 5700 0    50   ~ 0
-APOT11
+APOT21
 Text Label 13100 5900 0    50   ~ 0
-APOT11
+APOT22
 Text Label 15000 8200 2    50   ~ 0
 ALP31

Commit message: PCBv5 redesign current sensing
Parts:
- removed C11, C12, C22, C23: 0.1μF, Capacitor_SMD:C_0402_1005Metric, symbol EVE-PCB-V4-rescue:C-Device-EVE-PCB-rescue
- removed U10, U11, U15, U16: INA219AxDCN, Package_TO_SOT_SMD:SOT-23-8, symbol Analog_ADC:INA219AxDCN
- added C? (x4): 0.1μF, Capacitor_SMD:C_0402_1005Metric, symbol EVE-PCB-V4-rescue:C-Device-EVE-PCB-rescue
- added C? (x4): 1μF, Capacitor_SMD:C_0805_2012Metric, symbol EVE-PCB-V4-rescue:C-Device-EVE-PCB-rescue
- added R? (x4): 160KΩ, Resistor_SMD:R_0805_2012Metric, symbol EVE-PCB-V4-rescue:R-Device-EVE-PCB-rescue
- added R? (x2): 10KΩ, Resistor_SMD:R_0402_1005Metric, symbol EVE-PCB-V4-rescue:R-Device-EVE-PCB-rescue
- added U? (x2): LM2902, Package_SO:SOIC-14_3.9x8.7mm_P1.27mm, symbol Potentiometer_Digital:AD5254
- added U? (x5): LM2902, Package_SO:SOIC-14_3.9x8.7mm_P1.27mm, symbol Amplifier_Operational:LM2902
- added U?: LM2902, Package_SO:SOIC-14_3.9x8.7mm_P1.27mm, symbol EVE-PCB-V4-rescue:ADS1015IDGSR-ADS1015IDGSR
Connections:
- net +12V: now also C?.2, U?.17 (A3), U?.17 (A3), U?.4 (V+), U?.8 (A1), U?.8 (A1)
- net +5V: now also C?.1, C?.2, C?.2, R?.1, U?.20 (VDD), U?.20 (VDD), U?.4 (AD0), U?.8 (VDD)
- net FAN1_POS: now also R?.2
- net FAN2_POS: now also R?.2
- net FAN3_POS: now also R?.2
- net FAN4_POS: now also R?.2
- net GND: now also C?.1, C?.1, C?.1, C?.1, C?.1, C?.1, C?.1, C?.2, R?.2, U?.10 (VSS), U?.10 (VSS), U?.11 (V-), U?.15 (DGND), U?.15 (DGND), U?.16 (AD1), U?.16 (AD1), U?.18 (B3), U?.18 (B3), U?.3 (GND), U?.4 (AD0), U?.5 (~WP~), U?.5 (~WP~), U?.7 (B1), U?.7 (B1)
- net SDA-FAN: now reaches U22.15 (SD5)
- net SDA-FAN: now also U?.9 (SDA), U?.9 (SDA), U?.9 (SDA)
- net SCL-FAN: now reaches U22.16 (SC5)
- net SCL-FAN: now also U?.10 (SCL), U?.14 (SCL), U?.14 (SCL)
- new net: R?.2, U?.2 (ALERT/RDY)
- new net: R?.1, U?.1 (ADDR)
- new net FAN1_OAN: U?.1 (W0), U?.2 (-)
- new net FAN1_OAO: U?.1, U?.2 (B0), U?.4 (AIN0)
- new net FAN1_OAP: U?.3 (+), U?.6 (W1)
- new net FAN2_OAN: U?.13 (W2), U?.6 (-)
- new net FAN2_OAO: U?.12 (B2), U?.5 (AIN1), U?.7
- new net FAN2_OAP: U?.19 (W3), U?.5 (+)
- new net FAN3_OAN: U?.1 (W0), U?.9 (-)
- new net FAN3_OAO: U?.2 (B0), U?.6 (AIN2), U?.8
- new net FAN3_OAP: U?.10 (+), U?.6 (W1)
- new net FAN4_OAN: U?.13 (-), U?.13 (W2)
- new net FAN4_OAO: U?.12 (B2), U?.14, U?.7 (AIN3)
- new net FAN4_OAP: U?.12 (+), U?.19 (W3)
- new net FILT_FAN1: C?.2, R?.1, U?.3 (A0)
- new net FILT_FAN2: C?.2, R?.1, U?.11 (A2)
- new net FILT_FAN3: C?.2, R?.1, U?.3 (A0)
- new net FILT_FAN4: C?.2, R?.1, U?.11 (A2)
Other:
- moved on the sheet: R36, R37, R46, R47

Commit message: Updates to PCB v5
Parts:
- removed C? (x4): 0.1μF, Capacitor_SMD:C_0402_1005Metric, symbol EVE-PCB-V4-rescue:C-Device-EVE-PCB-rescue
- removed R? (x2): 10KΩ, Resistor_SMD:R_0402_1005Metric, symbol EVE-PCB-V4-rescue:R-Device-EVE-PCB-rescue
- removed U? (x2): LM2902, Package_SO:SOIC-14_3.9x8.7mm_P1.27mm, symbol Potentiometer_Digital:AD5254
- removed U? (x5): LM2902, Package_SO:SOIC-14_3.9x8.7mm_P1.27mm, symbol Amplifier_Operational:LM2902
- removed U?: LM2902, Package_SO:SOIC-14_3.9x8.7mm_P1.27mm, symbol EVE-PCB-V4-rescue:ADS1015IDGSR-ADS1015IDGSR
- added C22, C51, C52, C54: 0.1μF, Capacitor_SMD:C_0402_1005Metric, symbol EVE-PCB-V4-rescue:C-Device-EVE-PCB-rescue
- added U10, U11, U15, U32: INA219AxDCN, Package_TO_SOT_SMD:SOT-23-8, symbol Analog_ADC:INA219AxDCN
- R36, R37, R46, R47: value 0.4Ω -> 2.15Ω; footprint Resistor_SMD:R_2512_6332Metric -> Resistor_SMD:R_1206_3216Metric; LCSC C247521 -> C247507; Power 1.05 -> 0.077
- R75, R76, R77, R78: renamed from R?; value 160KΩ -> 750KΩ; footprint Resistor_SMD:R_0805_2012Metric -> Resistor_SMD:R_0603_1608Metric; LCSC C17485 -> C23240
- gave numbers to parts that had none: 4
Connections:
- net +12V: now also R75.2, R76.2, R77.2, R78.2
- net +5V: now also C22.1, C51.1, C52.1, C54.1, U10.4 (VS), U11.4 (VS), U11.7 (A0), U15.4 (VS), U15.8 (A1), U32.4 (VS), U32.7 (A0), U32.8 (A1)
- net FAN1_POS: now also C11.1, U10.2 (IN-); no longer R75.2
- net FAN2_POS: now also C12.1, U11.2 (IN-); no longer R76.2
- net FAN3_POS: now also C23.1, U15.2 (IN-); no longer R77.2
- net FAN4_POS: now also C50.1, U32.2 (IN-); no longer R78.2
- net FILT_FAN1: now also U10.1 (IN+)
- net FILT_FAN2: now also U11.1 (IN+)
- net FILT_FAN3: now also U15.1 (IN+)
- net FILT_FAN4: now also U32.1 (IN+)
- net GND: now also C22.2, C51.2, C52.2, C54.2, U10.3 (GND), U10.7 (A0), U10.8 (A1), U11.3 (GND), U11.8 (A1), U15.3 (GND), U15.7 (A0), U32.3 (GND); no longer C11.1, C12.1, C23.1, C50.1
- net SCL-CUR: now also U10.5 (SCL), U11.5 (SCL), U15.5 (SCL), U32.5 (SCL)
- net SDA-CUR: now also U10.6 (SDA), U11.6 (SDA), U15.6 (SDA), U32.6 (SDA)
- net SCL-FAN: no longer names the net of U22.16 (SC5)
- net SDA-FAN: no longer names the net of U22.15 (SD5)
Other:
- moved on the sheet: C23, C50, R46, R47, R77, R78
